File: pcb/servo_controller.brd (EAGLE design)
At the start: 68.6 x 53.3 mm, 31 parts, among them IC2 PIC18F452, U1 ARDUINOR3-DIMENSION

Commit message: Work
Parts:
- removed 6VOLTS: SE14, solpad:SE14
- added IC1: REG1117F, burr-brown:DD-3
- added R2, R3: (no value), rcl:M1206
- added S1: (no value), switch-omron:B3F-10XX
- moved C3 114.8 mm to (83.8, 72.4)
- moved C4 114.8 mm to (78.7, 72.4)
- moved C5 114.8 mm to (73.7, 72.4)
- moved C7 114.8 mm to (68.6, 72.4)
- moved C8 114.8 mm to (63.5, 72.4)
- moved DEBUG 114.8 mm to (83.8, 67.3)
- moved GND 114.8 mm to (69.8, 66.0)
- moved R1 114.8 mm to (88.9, 72.4)
- moved RX 114.8 mm to (97.8, 72.4)
- moved SCL 114.8 mm to (59.7, 66.0)
- moved SDA 114.8 mm to (64.8, 66.0)
- moved SV2 114.8 mm to (64.8, 61.0)
- moved TX 114.8 mm to (94.0, 72.4)
- moved X1 114.8 mm to (77.5, 40.6)
- moved SV3 49.6 mm to (30.5, 58.4)
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Connections:
- removed net N$29: 6VOLTS.MP
- removed net N$30: C3.1
- removed net N$40: C4.2
- removed net N$42: C3.2
- removed net N$43: GND.MP
- removed net VDDUC: C4.1
- new net +7V: C3.1, IC1.3, R2.2
- new net N$7: R2.1, R3.2
- net VSS: now also C3.2, GND.MP, IC1.1, R3.1

Commit message: Avancement carte électronique
Parts:
- removed X1: (no value), con-amp-micromatch:MICROMATCH-6
- added LED1, LED2: (no value), led:CHIPLED_0805
- added R4, R5, R6, R7: (no value), rcl:M0805
- added S2, S3: (no value), switch-omron:B3F-10XX
- added SV1: (no value), con-lsta:FE06
- S1: device switch-omron:B3F-10XX -> switch:255SB
- moved S1 13.1 mm to (5.08, 45.7), turned to 90 degrees
Connections:
- removed net RESET: IC2.18, R1.1, U1.RESET, X1.1
- new net LED0: LED1.C, U1.D8
- new net LED1: LED2.C, U1.D9
- new net LIPO_VOLTAGE: R2.1, R3.2, U1.A0
- new net N$8: LED2.A, R5.2
- new net SWITCH0: R7.1, S2.1, S2.2, U1.D10
- new net SWITCH1: R6.1, S3.1, S3.2, U1.D11
- new net UC_RESET: IC2.18, R1.1, SV1.1, U1.RESET
- new net VDD: C3.1, IC1.3, R2.2, S1.1
- net +5V: now also C4.1, IC1.2, R6.2, R7.2, SV1.2; no longer X1.2
- net +7V: now also S1.2; no longer C3.1, IC1.3, R2.2
- net N$22: now also SV1.4; no longer X1.4
- net N$23: now also SV1.5; no longer X1.5
- net N$7: now also LED1.A, R4.2; no longer R2.1, R3.2
- net VSS: now also C4.2, R4.1, R5.1, S2.3, S2.4, S3.3, S3.4, SV1.3; no longer X1.3

Commit message: Avancement PCB
Parts:
- removed GND: SE14, solpad:SE14
- removed SERVO12, SERVO13, SV2, SV3: (no value), con-lstb:MA03-1
- removed SV1: (no value), con-lsta:FE06
- added LIPO+, LIPO-: SE14, solpad:SE14
- added PGC, PGD, RESET, VDD, VSS: TPB1,27, testpad:B1,27
- added SERVO6, SERVO7, SERVOX, SERVOY: (no value), con-lstb:MA03-1
- added SV5: (no value), con-lstb:MA04-2
- DEBUG: device testpad:B2,54 -> testpad:B2,54@1
- moved C4 83.5 mm to (3.17, 36.8), flipped to the bottom, turned to 270 degrees
- moved C3 79.5 mm to (12.7, 36.8), flipped to the bottom, turned to 90 degrees
- moved R1 72.6 mm to (45.7, 14.0)
- moved C5 58.5 mm to (22.2, 44.5), turned to 270 degrees
- moved R2 53.8 mm to (54.0, 7.62), flipped to the bottom, turned to 180 degrees
- moved Q1 52.6 mm to (73.7, 45.7), flipped to the top, turned to 90 degrees
- moved R3 48.3 mm to (47.6, 7.62), flipped to the bottom, turned to 180 degrees
- moved DEBUG 47.7 mm to (48.3, 35.6)
- moved IC1 46.8 mm to (7.62, 27.3), flipped to the bottom, turned to 180 degrees
- moved RX 35.6 mm to (68.6, 52.1)
- moved TX 32.8 mm to (66.0, 55.2)
- moved C7 29.0 mm to (80.0, 45.7), turned to 90 degrees
- moved C8 27.5 mm to (78.7, 49.5), turned to 90 degrees
- moved SCL 12.0 mm to (53.3, 55.9)
- moved SERVO4 12.0 mm to (22.9, 34.3)
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Connections:
- removed net +7V: S1.2
- removed net N$20: SERVO10.2, SERVO11.2, SERVO12.2, SERVO13.2, SERVO8.2, SERVO9.2
- removed net N$21: SV3.2
- removed net N$26: SV2.2
- new net VEE: SERVO0.2, SERVO1.2, SERVO10.2, SERVO11.2, SERVO2.2, SERVO3.2, SERVO4.2, SERVO5.2, SERVO6.2, SERVO7.2, SERVO8.2, SERVO9.2, SERVOX.2, SERVOY.2
- net +5V: now also SV5.1, VDD.TP; no longer SV1.2
- net GND: now also SERVO6.1, SERVO7.1, SERVOX.1, SERVOY.1; no longer SERVO12.1, SERVO13.1, SV2.1, SV3.1
- net N$10: now also SERVO6.3; no longer SERVO8.3
- net N$11: now also SERVO7.3; no longer SERVO9.3
- net N$12: now also SERVO8.3; no longer SERVO10.3
- net N$13: now also SERVO9.3; no longer SERVO11.3
- net N$14: now also SERVO10.3; no longer SERVO12.3
- net N$15: now also LIPO+.MP, S1.2; no longer SERVO0.2, SERVO1.2, SERVO2.2, SERVO3.2, SERVO4.2, SERVO5.2
- net N$19: now also SERVOX.3; no longer SV2.3
- net N$22: now also PGD.TP; no longer SV1.4
- net N$23: now also PGC.TP; no longer SV1.5
- net N$24: now also SERVOY.3; no longer SV3.3
- net N$32: now also SERVO11.3; no longer SERVO13.3
- net UC_RESET: now also RESET.TP; no longer SV1.1
- net VSS: now also LIPO-.MP, SV5.2, VSS.TP; no longer GND.MP, SV1.3
Routing:
- net VEE: track 0.00 -> 86.1 mm
- net N$10: track 0.00 -> 18.0 mm
- net N$5: track 0.00 -> 17.9 mm
- net N$1: track 0.00 -> 17.8 mm
- net N$32: track 0.00 -> 16.9 mm
- net N$3: track 0.00 -> 16.0 mm
- net N$2: track 0.00 -> 15.9 mm
- net N$4: track 0.00 -> 14.7 mm
- net N$11: track 0.00 -> 14.6 mm
- net N$6: track 0.00 -> 14.5 mm
- net N$14: track 0.00 -> 13.7 mm
- net N$12: track 0.00 -> 10.0 mm
- net N$13: track 0.00 -> 8.69 mm
- net LIPO_VOLTAGE: track 0.00 -> 8.63 mm
- net N$24: track 0.00 -> 4.34 mm
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
Commit message: Pcb
Parts:
- added IC3: (no value), AWJLEagleLib:SO08
- PGC, PGD, RESET, VDD, VSS: value TPB1,27 -> TPTP20R; device testpad:B1,27 -> testpad:TP20R
- moved C7 49.4 mm to (32.7, 31.4), turned to 180 degrees
- moved Q1 39.2 mm to (39.4, 26.7), turned to 225 degrees
- moved C8 37.3 mm to (47.9, 28.6), flipped to the bottom
- moved C5 23.5 mm to (29.8, 22.2), turned to 90 degrees
- moved SCL 14.2 mm to (66.7, 51.1)
- moved SDA 12.8 mm to (67.0, 47.6)
- moved RX 12.1 mm to (67.3, 40.0)
- moved TX 11.5 mm to (67.0, 43.8)
- moved PGC 2.54 mm to (40.0, 8.89), flipped to the bottom
- moved PGD 2.01 mm to (37.5, 8.89), flipped to the bottom
- moved VSS 1.90 mm to (34.9, 8.89), flipped to the bottom
- moved VDD 1.27 mm to (32.4, 8.89), flipped to the bottom
- moved RESET 0.63 mm to (29.8, 8.89), flipped to the bottom
- moved SV5 0.63 mm to (64.1, 22.9)
- flipped R2 to the top, turned to 0 degrees
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Connections:
- new net SERVO_CURRENT: IC3.4, U1.A1
- net +5V: now also IC3.1
- net GND: no longer C8.2
- net VDD: now also IC3.8
- net VEE: now also IC3.6
- net VSS: now also C8.2, IC3.3
Routing:
- net N$25: track 0.00 -> 18.0 mm, vias 0 -> 1
- net VSS: track 0.00 -> 17.7 mm
- net +5V: track 0.00 -> 15.9 mm
- net N$27: track 0.00 -> 14.3 mm, vias 0 -> 1
- net LIPO_VOLTAGE: track 8.63 -> 0.00 mm
- net N$12: track 10.0 -> 15.4 mm
- net N$13: track 8.69 -> 14.0 mm
- net N$10: track 18.0 -> 21.3 mm
- net N$3: track 16.0 -> 17.9 mm
- net N$11: track 14.6 -> 16.4 mm
- net N$4: track 14.7 -> 15.9 mm
- net N$2: track 15.9 -> 16.6 mm

Commit message: Pcb
Parts:
- removed DEBUG: B2,54, testpad:B2,54@1
- removed R1: (no value), rcl:M1206
- SCL, SDA: value SE14 -> TPTP20R; device solpad:SE14 -> testpad:TP20R
- moved SERVO11 34.9 mm to (33.3, 40.6), turned to 270 degrees
- moved SCL 33.3 mm to (53.3, 20.6)
- moved SERVOX 30.9 mm to (62.2, 22.9), turned to 180 degrees
- moved SERVO10 29.6 mm to (37.1, 40.6), turned to 270 degrees
- moved SERVOY 25.5 mm to (62.2, 26.7), turned to 180 degrees
- moved SDA 25.1 mm to (53.3, 26.5)
- moved SERVO5 24.4 mm to (26.7, 14.0)
- moved C7 23.7 mm to (49.2, 14.4)
- moved SERVO0 21.9 mm to (26.7, 35.6)
- moved SERVO9 21.4 mm to (42.2, 40.6), turned to 270 degrees
- moved PGC 20.8 mm to (44.5, 29.2), turned to 270 degrees
- moved PGD 19.1 mm to (44.5, 26.7), turned to 270 degrees
- moved VSS 18.0 mm to (44.5, 24.1), turned to 270 degrees
- moved RESET 17.8 mm to (44.5, 19.1), turned to 270 degrees
- moved Q1 17.6 mm to (46.4, 10.5), turned to 180 degrees
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Connections:
- net +5V: no longer R1.2
- net GND: no longer C5.1, C7.1, SERVO0.1, SERVO1.1, SERVO10.1, SERVO11.1, SERVO2.1, SERVO3.1, SERVO4.1, SERVO5.1, SERVO6.1, SERVO7.1, SERVO8.1, SERVO9.1, SERVOX.1, SERVOY.1
- net N$17: no longer DEBUG.PP
- net N$18: now also SCL.TP; no longer SCL.MP
- net N$9: now also SDA.TP; no longer SDA.MP
- net UC_RESET: no longer R1.1
- net VSS: now also C5.1, C7.1, SERVO0.1, SERVO1.1, SERVO10.1, SERVO11.1, SERVO2.1, SERVO3.1, SERVO4.1, SERVO5.1, SERVO6.1, SERVO7.1, SERVO8.1, SERVO9.1, SERVOX.1, SERVOY.1
Routing:
- net VEE: track 86.1 -> 156.4 mm
- net UC_RESET: track 0.00 -> 17.2 mm, vias 0 -> 1
- net N$23: track 0.00 -> 15.7 mm, vias 0 -> 1
- net N$22: track 0.00 -> 14.9 mm, vias 0 -> 1
- net N$6: track 14.1 -> 25.4 mm, vias 0 -> 1
- net VSS: track 17.7 -> 26.2 mm
- net N$25: track 18.0 -> 11.2 mm, vias 1 -> 0
- net N$5: track 18.0 -> 11.7 mm
- net N$24: track 4.34 -> 10.5 mm
- net N$19: track 4.07 -> 9.64 mm
- net N$13: track 14.0 -> 8.91 mm
- net N$12: track 15.4 -> 11.0 mm
- net N$18: track 0.00 -> 3.88 mm
- net N$10: track 21.3 -> 17.6 mm
- net +5V: track 15.9 -> 19.4 mm
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- added copper zone on layer 1, net VSS
- added copper zone on layer 16, net VSS
- removed copper zone on layer 1, net GND
- removed copper zone on layer 16, net GND
Other:
- board text added: "Vérifier la taille des rivets"

Commit message: Pcb, encore !
Parts:
- removed IC1: REG1117F, burr-brown:DD-3
- removed RX, TX: SE14, solpad:SE14
- added IC4: LM2937, linear:TO263-3
- added R1: (no value), resistor-shunt:PMD
- C3: value (none) -> 100nf
- C4: value (none) -> 10uf
- moved LED1 28.0 mm to (19.1, 3.17), turned to 180 degrees
- moved LED2 27.5 mm to (21.6, 3.17), turned to 180 degrees
- moved IC3 23.8 mm to (6.03, 26.4), turned to 180 degrees
- moved R4 21.9 mm to (19.1, 7.62), turned to 90 degrees
- moved R5 21.2 mm to (21.6, 7.62), turned to 270 degrees
- moved C3 18.1 mm to (8.26, 45.1), turned to 180 degrees
- moved LIPO+ 4.45 mm to (3.17, 43.8)
- moved LIPO- 4.45 mm to (3.17, 39.4)
- moved C4 3.17 mm to (6.35, 33.0), turned to 180 degrees
Connections:
- removed net N$16: IC2.44, TX.MP
- removed net N$17: IC2.1, RX.MP
- new net RX_FROM_ARDUINO: IC2.44, U1.D0
- new net TX_FROM_ARDUINO: IC2.1, U1.D1
- net +5V: now also IC4.3; no longer IC1.2
- net VDD: now also IC4.1, R1.2; no longer IC1.3
- net VEE: now also R1.1
- net VSS: now also IC4.2; no longer IC1.1
Routing:
- net RX_FROM_ARDUINO: track 0.00 -> 31.6 mm
- net TX_FROM_ARDUINO: track 0.00 -> 30.5 mm
- net VSS: track 26.2 -> 23.8 mm
- net N$6: track 25.4 -> 26.6 mm
- net N$23: track 15.7 -> 16.4 mm

Commit message: PCB
Parts:
- removed SV5: (no value), con-lstb:MA04-2
- added C1: 100nf, rcl:C1206
- added D1: MBRA340T3, diode:SMA
- added SV1: (no value), con-lstb:MA03-2
- moved R2 13.7 mm to (47.6, 5.40), turned to 180 degrees
- moved R6 10.2 mm to (13.7, 16.5), turned to 270 degrees
- moved S2 8.57 mm to (7.30, 7.94)
- moved S3 7.62 mm to (7.30, 16.2), turned to 0 degrees
- moved R7 6.42 mm to (13.7, 7.94), turned to 90 degrees
- moved LED1 6.03 mm to (25.1, 3.17), turned to 0 degrees
- moved R4 5.85 mm to (22.9, 3.17), turned to 270 degrees
- moved R5 5.85 mm to (17.8, 3.17)
- moved C8 4.69 mm to (35.2, 11.4), turned to 270 degrees
- moved C4 3.59 mm to (3.81, 35.6)
- moved IC3 3.17 mm to (7.94, 23.8), turned to 270 degrees
- moved R3 2.71 mm to (54.0, 5.40), turned to 180 degrees
- moved R1 1.59 mm to (17.8, 24.1)
- moved LED2 1.59 mm to (20.0, 3.17), turned to 0 degrees
- moved C3 1.42 mm to (7.62, 43.8)
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Connections:
- new net N$20: C4.1, D1.A, IC4.3
- new net OPTION0: SV1.3, U1.A2
- new net OPTION1: SV1.5, U1.A3
- new net OPTION2: SV1.6, U1.A4
- new net OPTION3: SV1.4, U1.A5
- net +5V: now also C1.1, D1.C, SV1.1; no longer C4.1, IC4.3, SV5.1
- net SWITCH0: no longer S2.2
- net SWITCH1: no longer S3.1
- net VSS: now also C1.2, SV1.2; no longer SV5.2
Routing:
- net +5V: track 19.4 -> 120.7 mm, vias 0 -> 3
- net SERVO_CURRENT: track 0.00 -> 77.9 mm, vias 0 -> 1
- net SWITCH0: track 0.00 -> 74.9 mm
- net LED0: track 0.00 -> 66.3 mm, vias 0 -> 1
- net LED1: track 0.00 -> 64.2 mm, vias 0 -> 2
- net SWITCH1: track 0.00 -> 58.4 mm
- net VSS: track 23.8 -> 76.8 mm
- net VDD: track 0.00 -> 47.4 mm, vias 0 -> 1
- net UC_RESET: track 17.3 -> 38.0 mm, vias 1 -> 3
- net N$15: track 0.00 -> 17.6 mm
- net OPTION0: track 0.00 -> 12.0 mm
- net OPTION3: track 0.00 -> 12.0 mm
- net OPTION2: track 0.00 -> 7.62 mm
- net OPTION1: track 0.00 -> 7.62 mm
- net N$26: track 0.00 -> 6.35 mm
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Other:
- board text added: "Strap 0"
- board text removed: "Vérifier la taille des rivets"

Commit message: PCB
Parts:
- added C2: (no value), rcl:PANASONIC_D
- moved R5 2.54 mm to (20.3, 3.17)
- moved LED2 1.91 mm to (18.1, 3.17)
- moved C8 0.32 mm to (35.6, 11.4)
Connections:
- net VEE: now also C2.+
- net VSS: now also C2.-
Routing:
- net VSS: track 76.8 -> 163.7 mm, vias 0 -> 3
- net +5V: track 120.7 -> 151.1 mm, vias 3 -> 2
- net VEE: track 161.9 -> 170.1 mm, vias 0 -> 1
- net N$26: track 6.35 -> 0.00 mm
- net LED0: track 66.3 -> 70.8 mm
- net SWITCH0: track 74.9 -> 72.9 mm
- net LED1: track 64.2 -> 65.5 mm
- net N$8: track 2.87 -> 2.32 mm
Other:
- board text removed: "Strap 0"
