File: pcb/servo_controller.brd (EAGLE design)
At the start: 68.6 x 53.3 mm, 50 parts, among them IC2 PIC18F452, IC4 LM2937, U1 ARDUINOR3-DIMENSION

Commit message: Update
Routing:
- net +5V: track 153.6 -> 159.2 mm
Changed lines of the file:
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@@
 <plain>
 <text x="55.88" y="33.655" size="2.1844" layer="16" font="vector" rot="MR0">Vers. 1.0.1</text>
+<circle x="48.41875" y="28.09875" radius="0.15875" width="0.4064" layer="1"/>
 </plain>
 <attributes>
@@
 <contactref element="IC2" pad="44"/>
 <contactref element="U1" pad="D0"/>
-<wire x1="63.5" y1="50.8" x2="63.5" y2="48.26" width="0.6096" layer="1"/>
-<wire x1="63.5" y1="48.26" x2="62.23" y2="46.99" width="0.6096" layer="1"/>
-<wire x1="62.23" y1="46.99" x2="62.23" y2="35.56" width="0.6096" layer="1"/>
-<wire x1="62.23" y1="35.56" x2="57.15" y2="30.48" width="0.6096" layer="1"/>
-<wire x1="57.15" y1="30.48" x2="51.435" y2="30.48" width="0.6096" layer="1"/>
-<wire x1="51.435" y1="30.48" x2="50.165" y2="29.21" width="0.6096" layer="1"/>
-<wire x1="50.165" y1="29.21" x2="50.165" y2="28.2575" width="0.6096" layer="1"/>
 <wire x1="50.165" y1="28.2575" x2="50.25" y2="28.13" width="0.4064" layer="1"/>
+<wire x1="63.5" y1="50.8" x2="63.5" y2="48.26" width="0.4064" layer="1"/>
+<wire x1="63.5" y1="48.26" x2="62.23" y2="46.99" width="0.4064" layer="1"/>
+<wire x1="62.23" y1="46.99" x2="62.23" y2="35.56" width="0.4064" layer="1"/>
+<wire x1="62.23" y1="35.56" x2="57.15" y2="30.48" width="0.4064" layer="1"/>
+<wire x1="57.15" y1="30.48" x2="51.435" y2="30.48" width="0.4064" layer="1"/>
+<wire x1="51.435" y1="30.48" x2="50.165" y2="29.21" width="0.4064" layer="1"/>
+<wire x1="50.165" y1="29.21" x2="50.165" y2="28.215" width="0.4064" layer="1"/>
+<wire x1="50.165" y1="28.215" x2="50.25" y2="28.13" width="0.4064" layer="1"/>
 </signal>
 <signal name="TX_FROM_ARDUINO">
@@
 <wire x1="48.45" y1="29.93" x2="48.41875" y2="30.32125" width="0.4064" layer="1"/>
 <contactref element="U1" pad="D1"/>
-<wire x1="60.96" y1="50.8" x2="60.96" y2="36.195" width="0.6096" layer="1"/>
-<wire x1="60.96" y1="36.195" x2="56.515" y2="31.75" width="0.6096" layer="1"/>
-<wire x1="56.515" y1="31.75" x2="50.8" y2="31.75" width="0.6096" layer="1"/>
-<wire x1="50.8" y1="31.75" x2="48.895" y2="29.845" width="0.6096" layer="1"/>
 <wire x1="48.895" y1="29.845" x2="48.45" y2="29.93" width="0.4064" layer="1"/>
-<wire x1="48.895" y1="29.845" x2="48.5775" y2="29.845" width="0.6096" layer="1"/>
+<wire x1="60.96" y1="50.8" x2="60.96" y2="36.195" width="0.4064" layer="1"/>
+<wire x1="60.96" y1="36.195" x2="56.515" y2="31.75" width="0.4064" layer="1"/>
+<wire x1="56.515" y1="31.75" x2="50.8" y2="31.75" width="0.4064" layer="1"/>
+<wire x1="50.8" y1="31.75" x2="48.895" y2="29.845" width="0.4064" layer="1"/>
+<wire x1="48.895" y1="29.845" x2="48.535" y2="29.845" width="0.4064" layer="1"/>
+<wire x1="48.535" y1="29.845" x2="48.45" y2="29.93" width="0.4064" layer="1"/>
 </signal>
 <signal name="N$9">
@@
 <wire x1="37.7825" y1="25.7175" x2="38.6375" y2="25.7175" width="0.4064" layer="1"/>
 <wire x1="38.6375" y1="25.7175" x2="38.65" y2="25.73" width="0.4064" layer="1"/>
-<wire x1="33.3375" y1="38.1" x2="33.3375" y2="33.655" width="0.4064" layer="1"/>
-<wire x1="33.3375" y1="33.655" x2="37.1475" y2="29.845" width="0.4064" layer="1"/>
-<wire x1="37.1475" y1="29.845" x2="37.1475" y2="26.3525" width="0.4064" layer="1"/>
+<wire x1="33.3375" y1="38.1" x2="33.3375" y2="33.3375" width="0.4064" layer="1"/>
+<wire x1="33.3375" y1="33.3375" x2="37.1475" y2="29.5275" width="0.4064" layer="1"/>
+<wire x1="37.1475" y1="29.5275" x2="37.1475" y2="26.3525" width="0.4064" layer="1"/>
 <wire x1="37.1475" y1="26.3525" x2="37.7825" y2="25.7175" width="0.4064" layer="1"/>
 </signal>
@@
 <contactref element="IC2" pad="38"/>
 <wire x1="50.25" y1="23.33" x2="50.64125" y2="23.33625" width="0.4064" layer="1"/>
-<wire x1="50.64125" y1="23.33625" x2="52.3875" y2="23.33625" width="0.4064" layer="1"/>
-<wire x1="52.3875" y1="23.33625" x2="52.86375" y2="22.86" width="0.4064" layer="1"/>
-<wire x1="52.86375" y1="22.86" x2="59.69" y2="22.86" width="0.4064" layer="1"/>
+<wire x1="50.64125" y1="23.33625" x2="54.2925" y2="23.33625" width="0.4064" layer="1"/>
+<wire x1="54.2925" y1="23.33625" x2="54.76875" y2="22.86" width="0.4064" layer="1"/>
+<wire x1="54.76875" y1="22.86" x2="59.69" y2="22.86" width="0.4064" layer="1"/>
 </signal>
 <signal name="N$24">
@@
 <contactref element="IC3" pad="1"/>
 <contactref element="VDD" pad="TP"/>
-<wire x1="44.45" y1="18.33" x2="44.45" y2="23.33625" width="0.4064" layer="1"/>
-<wire x1="44.45" y1="23.33625" x2="43.65625" y2="24.13" width="0.4064" layer="1"/>
-<wire x1="43.65625" y1="24.13" x2="43.65625" y2="29.92375" width="0.4064" layer="1"/>
-<wire x1="43.65625" y1="29.92375" x2="43.65" y2="29.93" width="0.4064" layer="1"/>
+<wire x1="44.45" y1="18.33" x2="44.45" y2="19.685" width="0.4064" layer="1"/>
 <wire x1="44.45" y1="18.33" x2="44.45" y2="17.145" width="0.4064" layer="1"/>
 <wire x1="44.45" y1="17.145" x2="43.815" y2="16.51" width="0.4064" layer="1"/>
@@
 <wire x1="14.9225" y1="15.5575" x2="13.3375" y2="15.5575" width="0.6096" layer="1"/>
 <wire x1="13.3375" y1="15.5575" x2="13.6525" y2="15.56" width="0.6096" layer="1"/>
+<wire x1="44.45" y1="19.685" x2="44.1325" y2="20.0025" width="0.4064" layer="1"/>
+<wire x1="44.1325" y1="20.0025" x2="40.64" y2="20.0025" width="0.4064" layer="1"/>
+<wire x1="40.64" y1="20.0025" x2="40.3225" y2="20.32" width="0.4064" layer="1"/>
+<wire x1="40.3225" y1="20.32" x2="40.3225" y2="25.55875" width="0.4064" layer="1"/>
+<wire x1="40.3225" y1="25.55875" x2="41.5925" y2="26.82875" width="0.4064" layer="1"/>
+<wire x1="41.5925" y1="26.82875" x2="41.5925" y2="27.94" width="0.4064" layer="1"/>
+<wire x1="41.5925" y1="27.94" x2="41.91" y2="28.2575" width="0.4064" layer="1"/>
+<wire x1="41.91" y1="28.2575" x2="43.33875" y2="28.2575" width="0.4064" layer="1"/>
+<wire x1="43.33875" y1="28.2575" x2="43.65625" y2="28.575" width="0.4064" layer="1"/>
+<wire x1="43.65625" y1="28.575" x2="43.65625" y2="29.92375" width="0.4064" layer="1"/>
+<wire x1="43.65625" y1="29.92375" x2="43.65" y2="29.93" width="0.4064" layer="1"/>
 </signal>
 <signal name="GND">

Commit message: Modif pcb
Routing:
- net N$16: track 0.00 -> 239.9 mm
- net N$17: track 0.00 -> 239.9 mm
- net VDD: track 50.0 -> 139.9 mm, vias 1 -> 2
- net VSS: track 213.3 -> 240.4 mm
- net SERVO_CURRENT: track 78.3 -> 80.3 mm
- net N$15: track 17.6 -> 15.5 mm
- net SWITCH0: track 71.4 -> 72.0 mm
- net SWITCH1: track 59.0 -> 58.4 mm
- net UC_RESET: track 38.5 -> 38.0 mm

Commit message: Rev. 1.0.2, gerber file generation
Parts:
- removed IC4: LM2937, linear:TO263-3
- removed LED2: (no value), led:CHIPLED_0805
- removed LIPO+, LIPO-: SE14, solpad:SE14
- removed R7: (no value), rcl:M0805
- removed S3: (no value), switch-omron:B3F-10XX
- added IC1: PIC18F452, microchip:TQFP44
- added LED0: (no value), led:CHIPLED_0805
- added R1: (no value), rcl:M1206
- added SP: (no value), switch:255SB
- added X1: (no value), con-wago-500:W237-102
- C2: value (none) -> 10uf; device rcl:PANASONIC_D -> rcl:C1206
- C4: value 10uf -> (none); device rcl:C1206 -> rcl:PANASONIC_D
- C5: device rcl:C1206 -> rcl:PANASONIC_D
- C6: device rcl:PANASONIC_D -> rcl:C1206
- IC2: value PIC18F452 -> LM2936MP-3.0; device microchip:TQFP44 -> national-semiconductor:SOT223
- R3: device rcl:M1206 -> rcl:M0805
- S1: device switch:255SB -> switch-omron:B3F-10XX
- moved S1 34.3 mm to (7.30, 15.2), turned to 0 degrees
- moved IC2 31.4 mm to (15.9, 37.1)
- moved R3 31.2 mm to (22.9, 3.17), turned to 270 degrees
- moved C6 31.0 mm to (35.6, 11.4), turned to 270 degrees
- moved C5 25.6 mm to (18.1, 12.4), turned to 45 degrees
- moved C2 25.1 mm to (3.81, 33.0), turned to 180 degrees
- moved C4 24.2 mm to (27.3, 41.3), turned to 315 degrees
- moved C1 17.5 mm to (14.3, 42.5), turned to 0 degrees
- moved C3 15.7 mm to (3.81, 28.6), turned to 90 degrees
- moved R5 14.9 mm to (13.7, 16.5)
- moved C8 14.0 mm to (49.2, 14.4), turned to 180 degrees
- moved R6 8.57 mm to (13.7, 7.94), turned to 90 degrees
- moved LED1 6.98 mm to (18.1, 3.17)
- moved R2 6.38 mm to (54.0, 6.03)
- moved C7 5.56 mm to (43.7, 14.4), turned to 0 degrees
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- renumbered S2 to S0, SERVO0 to SRV0, SERVO1 to SRV1, SERVO10 to SRV10, SERVO11 to SRV11, SERVO2 to SRV2, SERVO3 to SRV3, SERVO4 to SRV4, SERVO5 to SRV5, SERVO6 to SRV6, SERVO7 to SRV7, SERVO8 to SRV8, SERVO9 to SRV9, SERVOX to SRVX, SERVOY to SRVY
Connections:
- removed net N$8 (its old number): LED2.A, R5.2
- new net N$7: LED0.A, R3.2
- net +5V: now also C3.1, C6.1, IC1.28, IC1.7, R5.2; no longer C1.1, C8.1, IC2.28, IC2.7, R7.2
- net LED0: now also LED0.C; no longer LED1.C
- net LED1: now also LED1.C; no longer LED2.C
- net LIPO_VOLTAGE: now also R1.1, R2.2; no longer R2.1, R3.2
- net N$1: now also IC1.19; no longer IC2.19
- net N$10: now also IC1.8; no longer IC2.8
- net N$11: now also IC1.9; no longer IC2.9
- net N$12: now also IC1.10; no longer IC2.10
- net N$13: now also IC1.11; no longer IC2.11
- net N$14: now also IC1.14; no longer IC2.14
- net N$15: now also SP.2, X1.2; no longer LIPO+.MP, S1.2
- net N$18: now also IC1.37; no longer IC2.37
- net N$19: now also IC1.38; no longer IC2.38
- net N$2: now also IC1.20; no longer IC2.20
- net N$20: now also C2.1, IC2.3; no longer C4.1, IC4.3
- net N$22: now also IC1.17; no longer IC2.17
- net N$23: now also IC1.16; no longer IC2.16
- net N$24: now also IC1.39; no longer IC2.39
- net N$25: now also C8.2, IC1.31; no longer C7.2, IC2.31
- net N$27: now also C7.2, IC1.30; no longer C5.2, IC2.30
- net N$3: now also IC1.21; no longer IC2.21
- net N$32: now also IC1.15; no longer IC2.15
- net N$4: now also IC1.22; no longer IC2.22
- net N$5: now also IC1.23; no longer IC2.23
- net N$6: now also IC1.32; no longer IC2.32
- net N$9: now also IC1.42; no longer IC2.42
- net RX_FROM_ARDUINO: now also IC1.44; no longer IC2.44
- net SWITCH0: now also R6.1; no longer R7.1
- net SWITCH1: now also R5.1, S1.2; no longer R6.1, S3.2
- net TX_FROM_ARDUINO: now also IC1.1; no longer IC2.1
- net UC_RESET: now also IC1.18; no longer IC2.18
- net VDD: now also C1.1, IC2.1, R1.2, SP.1; no longer C3.1, IC4.1, R2.2, S1.1
- net VEE: now also C4.+, C5.+; no longer C2.+, C6.+
- net VSS: now also C2.2, C4.-, C5.-, C6.2, C8.1, IC1.29, IC1.6, IC2.2, IC2.4, R2.1, S1.3, S1.4, X1.1; no longer C2.-, C4.2, C5.1, C6.-, C8.2, IC2.29, IC2.6, IC4.2, LIPO-.MP, R5.1, S3.3, S3.4
Routing:
- net N$16: track 239.9 -> 0.00 mm
- net N$17: track 239.9 -> 0.00 mm
- net VSS: track 240.4 -> 193.2 mm, vias 4 -> 3
- net N$20: track 5.49 -> 9.11 mm
- net VDD: track 139.9 -> 142.3 mm
- net N$8 (its old number): track 2.32 -> 0.00 mm
- net N$7: track 0.00 -> 2.32 mm
- net N$15: track 15.5 -> 13.8 mm
- net LIPO_VOLTAGE: track 6.30 -> 6.93 mm
Other:
- board text added: "+"
- board text added: "-"
- board text added: "Bleuette"
- board text added: "ON"
- board text added: "Rev. 1.0.2"
- board text added: "Servo controller"
- board text removed: "Vers. 1.0.1"

Commit message: Set values
Parts:
- C6: value (none) -> 100nf
- C7, C8: value (none) -> 22pf
- Q1: value (none) -> 10Mhz
- R1: value (none) -> 3.3k
- R2: value (none) -> 10k
- R3, R4: value (none) -> 1k
- R5, R6: value (none) -> 2.2k
Changed lines of the file:
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@@
 </autorouter>
 <elements>
-<element name="Q1" library="crystal" package="HC49UP" value="" x="46.355" y="10.4775" smashed="yes" rot="R180">
+<element name="Q1" library="crystal" package="HC49UP" value="10Mhz" x="46.355" y="10.4775" smashed="yes" rot="R180">
 <attribute name="NAME" x="54.9275" y="13.3985" size="1.27" layer="25" ratio="10" rot="R180"/>
 <attribute name="VALUE" x="52.07" y="14.6685" size="1.27" layer="27" ratio="10" rot="R180"/>
@@
 <attribute name="VALUE" x="66.04" y="29.591" size="1.27" layer="27" ratio="10" rot="R180"/>
 </element>
-<element name="C7" library="rcl" package="C1206" value="" x="43.65625" y="14.44625" smashed="yes">
+<element name="C7" library="rcl" package="C1206" value="22pf" x="43.65625" y="14.44625" smashed="yes">
 <attribute name="NAME" x="41.75125" y="15.58925" size="1.27" layer="25"/>
 <attribute name="VALUE" x="42.38625" y="12.03325" size="1.27" layer="27"/>
 </element>
-<element name="C8" library="rcl" package="C1206" value="" x="49.2125" y="14.44625" smashed="yes" rot="R180">
+<element name="C8" library="rcl" package="C1206" value="22pf" x="49.2125" y="14.44625" smashed="yes" rot="R180">
 <attribute name="NAME" x="48.895" y="16.79575" size="1.27" layer="25" rot="R180"/>
 <attribute name="VALUE" x="50.4825" y="16.85925" size="1.27" layer="27" rot="R180"/>
 </element>
-<element name="C6" library="rcl" package="C1206" value="" x="35.56" y="11.43" smashed="yes" rot="R270">
+<element name="C6" library="rcl" package="C1206" value="100nf" x="35.56" y="11.43" smashed="yes" rot="R270">
 <attribute name="NAME" x="36.83" y="12.2555" size="1.27" layer="25"/>
 <attribute name="VALUE" x="33.147" y="12.7" size="1.27" layer="27" rot="R270"/>
 </element>
 <element name="U1" library="adafruit" package="ARDUINOR3" value="ARDUINOR3-DIMENSION" x="0" y="0"/>
-<element name="R1" library="rcl" package="M1206" value="" x="47.625" y="6.0325" smashed="yes" rot="R180">
+<element name="R1" library="rcl" package="M1206" value="3.3k" x="47.625" y="6.0325" smashed="yes" rot="R180">
 <attribute name="NAME" x="45.085" y="6.6675" size="1.27" layer="25" rot="R180"/>
 <attribute name="VALUE" x="48.895" y="8.5725" size="1.27" layer="27" rot="R180"/>
 </element>
-<element name="R2" library="rcl" package="M1206" value="" x="53.975" y="6.0325" smashed="yes" rot="R180">
+<element name="R2" library="rcl" package="M1206" value="10k" x="53.975" y="6.0325" smashed="yes" rot="R180">
 <attribute name="NAME" x="58.42" y="6.6675" size="1.27" layer="25" rot="R180"/>
 <attribute name="VALUE" x="55.245" y="8.5725" size="1.27" layer="27" rot="R180"/>
@@
 <attribute name="VALUE" x="20.6375" y="1.905" size="1.27" layer="27" rot="R90"/>
 </element>
-<element name="R3" library="rcl" package="M0805" value="" x="22.86" y="3.175" smashed="yes" rot="R270">
+<element name="R3" library="rcl" package="M0805" value="1k" x="22.86" y="3.175" smashed="yes" rot="R270">
 <attribute name="NAME" x="21.9075" y="5.3975" size="1.27" layer="25"/>
 <attribute name="VALUE" x="20.32" y="4.445" size="1.27" layer="27" rot="R270"/>
 </element>
-<element name="R4" library="rcl" package="M0805" value="" x="20.32" y="3.175" smashed="yes" rot="R270">
+<element name="R4" library="rcl" package="M0805" value="1k" x="20.32" y="3.175" smashed="yes" rot="R270">
 <attribute name="NAME" x="19.05" y="5.3975" size="1.27" layer="25"/>
 <attribute name="VALUE" x="17.78" y="4.445" size="1.27" layer="27" rot="R270"/>
 </element>
-<element name="R5" library="rcl" package="M0805" value="" x="13.6525" y="16.51" smashed="yes" rot="R270">
+<element name="R5" library="rcl" package="M0805" value="2.2k" x="13.6525" y="16.51" smashed="yes" rot="R270">
 <attribute name="NAME" x="12.3825" y="18.415" size="1.27" layer="25"/>
 <attribute name="VALUE" x="11.1125" y="17.78" size="1.27" layer="27" rot="R270"/>
 </element>
-<element name="R6" library="rcl" package="M0805" value="" x="13.6525" y="7.9375" smashed="yes" rot="R90">
+<element name="R6" library="rcl" package="M0805" value="2.2k" x="13.6525" y="7.9375" smashed="yes" rot="R90">
 <attribute name="NAME" x="16.8275" y="8.5725" size="1.27" layer="25" rot="R180"/>
 <attribute name="VALUE" x="16.1925" y="6.6675" size="1.27" layer="27" rot="R90"/>
