File: pcb/servo_controller.sch (EAGLE design)
At the start: 31 parts, among them IC2 PIC18F452, U1 ARDUINOR3-DIMENSION

Commit message: Work
Parts:
- removed 6VOLTS: SE14, solpad:SE14
- added IC1: REG1117F, burr-brown:REG1117F
- added R2, R3: (no value), rcl:R-EU_M1206
- added S1: (no value), switch-omron:10-XX
Connections:
- removed net N$29: 6VOLTS.MP
- removed net N$30: C3.1
- removed net N$40: C4.2
- removed net N$42: C3.2
- removed net N$43: GND.MP
- removed net VDDUC: C4.1
- new net +7V: C3.1, IC1.VIN, R2.2
- new net N$7: R2.1, R3.2
- net VSS: now also C3.2, GND.MP, IC1.GND, R3.1
Other:
- moved on the sheet: C3, C4, GND

Commit message: Avancement carte électronique
Parts:
- removed X1: (no value), con-amp-micromatch:MICROMATCH-6
- added LED1, LED2: (no value), led:LEDCHIPLED_0805
- added R4, R5, R6, R7: (no value), rcl:R-EU_M0805
- added S2, S3: (no value), switch-omron:10-XX
- added SV1: (no value), con-lsta:FE06-1
- S1: device switch-omron:10-XX -> switch:255SB
Connections:
- removed net RESET: IC2.!MCLR/THV, R1.1, U1./RESET, X1-1.S
- new net LED0: LED1.C, U1.D8
- new net LED1: LED2.C, U1.D9
- new net LIPO_VOLTAGE: R2.1, R3.2, U1.A0
- new net N$8: LED2.A, R5.2
- new net SWITCH0: R7.1, S2.S, S2.S1, U1.D10
- new net SWITCH1: R6.1, S3.S, S3.S1, U1.D11
- new net UC_RESET: IC2.!MCLR/THV, R1.1, SV1.1, U1./RESET
- new net VDD: C3.1, IC1.VIN, R2.2, S1.O
- net +5V: now also C4.1, IC1.VOUT, R6.2, R7.2, SV1.2; no longer X1-2.S
- net +7V: now also S1.P; no longer C3.1, IC1.VIN, R2.2
- net N$22: now also SV1.4; no longer X1-4.S
- net N$23: now also SV1.5; no longer X1-5.S
- net N$7: now also LED1.A, R4.2; no longer R2.1, R3.2
- net VSS: now also C4.2, R4.1, R5.1, S2.P, S2.P1, S3.P, S3.P1, SV1.3; no longer X1-3.S
Other:
- moved on the sheet: C3, C4, GND

Commit message: Avancement PCB
Parts:
- removed SERVO12, SERVO13: (no value), con-lstb:MA03-1
- removed SV1: (no value), con-lsta:FE06-1
- added LIPO+: SE14, solpad:SE14
- added PGC, PGD, RESET, VDD, VSS: TPB1,27, testpad:TPB1,27
- added SERVO6, SERVO7: (no value), con-lstb:MA03-1
- added SV5: (no value), con-lstb:MA04-2
- renumbered GND to LIPO-, SV2 to SERVOX, SV3 to SERVOY
Connections:
- removed net +7V: S1.P
- removed net N$20: SERVO10.2, SERVO11.2, SERVO12.2, SERVO13.2, SERVO8.2, SERVO9.2
- removed net N$21: SERVOY.2
- removed net N$26: SERVOX.2
- new net VEE: SERVO0.2, SERVO1.2, SERVO10.2, SERVO11.2, SERVO2.2, SERVO3.2, SERVO4.2, SERVO5.2, SERVO6.2, SERVO7.2, SERVO8.2, SERVO9.2, SERVOX.2, SERVOY.2
- net +5V: now also SV5.1, VDD.TP; no longer SV1.2
- net GND: now also SERVO6.1, SERVO7.1; no longer SERVO12.1, SERVO13.1
- net N$10: now also SERVO6.3; no longer SERVO8.3
- net N$11: now also SERVO7.3; no longer SERVO9.3
- net N$12: now also SERVO8.3; no longer SERVO10.3
- net N$13: now also SERVO9.3; no longer SERVO11.3
- net N$14: now also SERVO10.3; no longer SERVO12.3
- net N$15: now also LIPO+.MP, S1.P; no longer SERVO0.2, SERVO1.2, SERVO2.2, SERVO3.2, SERVO4.2, SERVO5.2
- net N$22: now also PGD.TP; no longer SV1.4
- net N$23: now also PGC.TP; no longer SV1.5
- net N$32: now also SERVO11.3; no longer SERVO13.3
- net UC_RESET: now also RESET.TP; no longer SV1.1
- net VSS: now also SV5.2, VSS.TP; no longer SV1.3
Other:
- moved on the sheet: LED1, LED2, R4, R5, R6, R7, S2, S3, SERVO10, SERVO11, SERVO8, SERVO9

Commit message: Pcb
Parts:
- added IC3: (no value), AWJLEagleLib:MAX4173A
- PGC, PGD, RESET, VDD, VSS: value TPB1,27 -> TPTP20R; device testpad:TPB1,27 -> testpad:TPTP20R
Connections:
- new net SERVO_CURRENT: IC3.VOUT, U1.A1
- net +5V: now also IC3.VCC
- net GND: no longer C8.2
- net VDD: now also IC3.R+
- net VEE: now also IC3.R-
- net VSS: now also C8.2, IC3.GND
Other:
- moved on the sheet: R2, R3
Changed lines of the file:
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@@
 <setting verticaltext="up"/>
 </settings>
-<grid distance="0.1" unitdist="inch" unit="inch" style="dots" multiple="1" display="yes" altdistance="0.025" altunitdist="inch" altunit="inch"/>
+<grid distance="0.1" unitdist="inch" unit="inch" style="dots" multiple="1" display="yes" altdistance="0.01" altunitdist="inch" altunit="inch"/>
 <layers>
 <layer number="1" name="Top" color="4" fill="1" visible="no" active="no"/>
@@
 <part name="GND6" library="supply1" deviceset="GND" device=""/>
 <part name="GND8" library="supply1" deviceset="GND" device=""/>
-<part name="GND9" library="supply1" deviceset="GND" device=""/>
 <part name="IC1" library="burr-brown" deviceset="REG1117" device="F"/>
 <part name="VSS3" library="supply1" deviceset="VSS" device=""/>
@@
 <part name="LIPO+" library="solpad" deviceset="SE14" device=""/>
 <part name="LIPO-" library="solpad" deviceset="SE14" device=""/>
-<part name="RESET" library="testpad" deviceset="TP" device="B1,27"/>
-<part name="VDD" library="testpad" deviceset="TP" device="B1,27"/>
-<part name="VSS" library="testpad" deviceset="TP" device="B1,27"/>
-<part name="PGD" library="testpad" deviceset="TP" device="B1,27"/>
-<part name="PGC" library="testpad" deviceset="TP" device="B1,27"/>
+<part name="IC3" library="AWJLEagleLib" deviceset="MAX4173" device="A"/>
+<part name="VSS14" library="supply1" deviceset="VSS" device=""/>
+<part name="VDD2" library="supply1" deviceset="VDD" device="" value="LIPO"/>
+<part name="RESET" library="testpad" deviceset="TP" device="TP20R"/>
+<part name="VDD" library="testpad" deviceset="TP" device="TP20R"/>
+<part name="VSS" library="testpad" deviceset="TP" device="TP20R"/>
+<part name="PGD" library="testpad" deviceset="TP" device="TP20R"/>
+<part name="PGC" library="testpad" deviceset="TP" device="TP20R"/>
+<part name="SUPPLY5" library="supply2" deviceset="VEE" device="" value="SERVO"/>
+<part name="VSS16" library="supply1" deviceset="VSS" device=""/>
 </parts>
 <sheets>
@@
 <instance part="GND6" gate="1" x="60.96" y="60.96"/>
 <instance part="GND8" gate="1" x="264.16" y="43.18"/>
-<instance part="GND9" gate="1" x="124.46" y="106.68"/>
 <instance part="IC1" gate="G$1" x="96.52" y="236.22"/>
 <instance part="VSS3" gate="G$1" x="27.94" y="220.98"/>
 <instance part="VSS4" gate="G$1" x="81.28" y="220.98"/>
 <instance part="VSS5" gate="G$1" x="96.52" y="220.98"/>
-<instance part="R2" gate="G$1" x="48.26" y="208.28" rot="R90"/>
-<instance part="R3" gate="G$1" x="48.26" y="193.04" rot="R90"/>
-<instance part="VSS6" gate="G$1" x="48.26" y="182.88"/>
+<instance part="R2" gate="G$1" x="48.26" y="228.6" rot="R90"/>
+<instance part="R3" gate="G$1" x="48.26" y="213.36" rot="R90"/>
+<instance part="VSS6" gate="G$1" x="48.26" y="203.2"/>
 <instance part="S1" gate="1" x="35.56" y="236.22" rot="R270"/>
 <instance part="P+1" gate="1" x="111.76" y="241.3"/>
-<instance part="P+8" gate="1" x="111.76" y="175.26"/>
+<instance part="P+8" gate="1" x="38.1" y="177.8"/>
 <instance part="P+9" gate="1" x="124.46" y="177.8"/>
 <instance part="P+10" gate="1" x="134.62" y="175.26"/>
@@
 <instance part="LIPO+" gate="1" x="22.86" y="233.68" rot="R90"/>
 <instance part="LIPO-" gate="1" x="22.86" y="226.06" rot="R90"/>
+<instance part="IC3" gate="G$1" x="55.88" y="172.72"/>
+<instance part="VSS14" gate="G$1" x="38.1" y="162.56"/>
+<instance part="VDD2" gate="G$1" x="38.1" y="193.04"/>
 <instance part="RESET" gate="G$1" x="104.14" y="149.86" smashed="yes">
-<attribute name="NAME" x="104.14" y="151.13" size="1.778" layer="95" rot="R90"/>
+<attribute name="NAME" x="104.775" y="151.13" size="1.778" layer="95" rot="R90"/>
 <attribute name="TP_SIGNAL_NAME" x="105.41" y="148.59" size="1.778" layer="97"/>
 </instance>
 <instance part="VDD" gate="G$1" x="106.68" y="149.86" smashed="yes">
-<attribute name="NAME" x="106.68" y="151.13" size="1.778" layer="95" rot="R90"/>
+<attribute name="NAME" x="107.315" y="151.13" size="1.778" layer="95" rot="R90"/>
 <attribute name="TP_SIGNAL_NAME" x="107.95" y="148.59" size="1.778" layer="97"/>
 </instance>
 <instance part="VSS" gate="G$1" x="109.22" y="149.86" smashed="yes">
-<attribute name="NAME" x="109.22" y="151.13" size="1.778" layer="95" rot="R90"/>
+<attribute name="NAME" x="109.855" y="151.13" size="1.778" layer="95" rot="R90"/>
 <attribute name="TP_SIGNAL_NAME" x="110.49" y="148.59" size="1.778" layer="97"/>
 </instance>
 <instance part="PGD" gate="G$1" x="111.76" y="149.86" smashed="yes">
-<attribute name="NAME" x="111.76" y="151.13" size="1.778" layer="95" rot="R90"/>
+<attribute name="NAME" x="112.395" y="151.13" size="1.778" layer="95" rot="R90"/>
 <attribute name="TP_SIGNAL_NAME" x="113.03" y="148.59" size="1.778" layer="97"/>
 </instance>
 <instance part="PGC" gate="G$1" x="114.3" y="149.86" smashed="yes">
-<attribute name="NAME" x="114.3" y="151.13" size="1.778" layer="95" rot="R90"/>
+<attribute name="NAME" x="114.935" y="151.13" size="1.778" layer="95" rot="R90"/>
 <attribute name="TP_SIGNAL_NAME" x="115.57" y="148.59" size="1.778" layer="97"/>
 </instance>
+<instance part="SUPPLY5" gate="G$1" x="73.66" y="193.04"/>
+<instance part="VSS16" gate="G$1" x="124.46" y="106.68"/>
 </instances>
 <busses>
@@
 <pinref part="R3" gate="G$1" pin="1"/>
 <pinref part="VSS6" gate="G$1" pin="VSS"/>
-<wire x1="48.26" y1="185.42" x2="48.26" y2="187.96" width="0.1524" layer="91"/>
+<wire x1="48.26" y1="205.74" x2="48.26" y2="208.28" width="0.1524" layer="91"/>
 </segment>
 <segment>
@@
 <pinref part="VSS13" gate="G$1" pin="VSS"/>
 <wire x1="177.8" y1="167.64" x2="177.8" y2="165.1" width="0.1524" layer="91"/>
+</segment>
+<segment>
+<pinref part="IC3" gate="G$1" pin="GND"/>
+<wire x1="40.64" y1="167.64" x2="38.1" y2="167.64" width="0.1524" layer="91"/>
+<pinref part="VSS14" gate="G$1" pin="VSS"/>
+<wire x1="38.1" y1="167.64" x2="38.1" y2="165.1" width="0.1524" layer="91"/>
+</segment>
+<segment>
+<wire x1="121.285" y1="111.76" x2="124.46" y2="111.76" width="0.1524" layer="91"/>
+<wire x1="124.46" y1="111.76" x2="124.46" y2="109.22" width="0.1524" layer="91"/>
+<pinref part="C8" gate="G$1" pin="2"/>
+<pinref part="VSS16" gate="G$1" pin="VSS"/>
 </segment>
 </net>
@@
 <pinref part="P+11" gate="1" pin="+5V"/>
 <wire x1="198.12" y1="167.64" x2="198.12" y2="180.34" width="0.1524" layer="91"/>
+</segment>
+<segment>
+<pinref part="IC3" gate="G$1" pin="VCC"/>
+<wire x1="40.64" y1="172.72" x2="38.1" y2="172.72" width="0.1524" layer="91"/>
+<pinref part="P+8" gate="1" pin="+5V"/>
+<wire x1="38.1" y1="172.72" x2="38.1" y2="175.26" width="0.1524" layer="91"/>
 </segment>
 </net>
@@
 <pinref part="GND6" gate="1" pin="GND"/>
 </segment>
-<segment>
-<wire x1="121.285" y1="111.76" x2="124.46" y2="111.76" width="0.1524" layer="91"/>
-<wire x1="124.46" y1="111.76" x2="124.46" y2="109.22" width="0.1524" layer="91"/>
-<pinref part="C8" gate="G$1" pin="2"/>
-<pinref part="GND9" gate="1" pin="GND"/>
-</segment>
 </net>
 <net name="VDD" class="0">
@@
 <junction x="81.28" y="236.22"/>
 <pinref part="R2" gate="G$1" pin="2"/>
-<wire x1="48.26" y1="236.22" x2="48.26" y2="213.36" width="0.1524" layer="91"/>
+<wire x1="48.26" y1="236.22" x2="48.26" y2="233.68" width="0.1524" layer="91"/>
 <pinref part="S1" gate="1" pin="O"/>
 <wire x1="40.64" y1="236.22" x2="48.26" y2="236.22" width="0.1524" layer="91"/>
@@
 <wire x1="48.26" y1="236.22" x2="48.26" y2="238.76" width="0.1524" layer="91"/>
 </segment>
+<segment>
+<pinref part="VDD2" gate="G$1" pin="VDD"/>
+<wire x1="38.1" y1="190.5" x2="38.1" y2="187.96" width="0.1524" layer="91"/>
+<wire x1="38.1" y1="187.96" x2="48.26" y2="187.96" width="0.1524" layer="91"/>
+<pinref part="IC3" gate="G$1" pin="R+"/>
+<wire x1="48.26" y1="187.96" x2="48.26" y2="185.42" width="0.1524" layer="91"/>
+</segment>
 </net>
 <net name="N$7" class="0">
@@
 <pinref part="R2" gate="G$1" pin="1"/>
 <pinref part="R3" gate="G$1" pin="2"/>
-<wire x1="48.26" y1="198.12" x2="48.26" y2="200.66" width="0.1524" layer="91"/>
-<wire x1="48.26" y1="200.66" x2="48.26" y2="203.2" width="0.1524" layer="91"/>
-<wire x1="48.26" y1="200.66" x2="60.96" y2="200.66" width="0.1524" layer="91"/>
-<label x="63.5" y="200.66" size="1.778" layer="95"/>
-<junction x="48.26" y="200.66"/>
-<junction x="60.96" y="200.66"/>
+<wire x1="48.26" y1="218.44" x2="48.26" y2="220.98" width="0.1524" layer="91"/>
+<wire x1="48.26" y1="220.98" x2="48.26" y2="223.52" width="0.1524" layer="91"/>
+<wire x1="48.26" y1="220.98" x2="53.34" y2="220.98" width="0.1524" layer="91"/>
+<label x="55.88" y="220.98" size="1.778" layer="95"/>
+<junction x="48.26" y="220.98"/>
+<junction x="53.34" y="220.98"/>
 </segment>
 </net>
@@
 <pinref part="SUPPLY4" gate="G$1" pin="VEE"/>
 </segment>
+<segment>
+<pinref part="IC3" gate="G$1" pin="R-"/>
+<wire x1="63.5" y1="185.42" x2="63.5" y2="187.96" width="0.1524" layer="91"/>
+<wire x1="63.5" y1="187.96" x2="73.66" y2="187.96" width="0.1524" layer="91"/>
+<pinref part="SUPPLY5" gate="G$1" pin="VEE"/>
+<wire x1="73.66" y1="187.96" x2="73.66" y2="190.5" width="0.1524" layer="91"/>
+</segment>
 </net>
 <net name="N$15" class="0">
@@
 </segment>
 </net>
+<net name="SERVO_CURRENT" class="0">
+<segment>
+<pinref part="IC3" gate="G$1" pin="VOUT"/>
+<wire x1="71.12" y1="170.18" x2="73.66" y2="170.18" width="0.1524" layer="91"/>
+<junction x="73.66" y="170.18"/>
+<label x="76.2" y="170.18" size="1.778" layer="95"/>
+</segment>
+<segment>
+<pinref part="U1" gate="G$1" pin="A1"/>
+<wire x1="287.02" y1="154.94" x2="287.02" y2="142.24" width="0.1524" layer="91"/>
+<junction x="287.02" y="142.24"/>
+<label x="287.02" y="119.38" size="1.778" layer="95" rot="R90"/>
+</segment>
+</net>

Commit message: Pcb
Parts:
- removed DEBUG: B2,54, testpad:B2,54
- removed R1: (no value), rcl:R-EU_M1206
- SCL, SDA: value SE14 -> TPTP20R; device solpad:SE14 -> testpad:TPTP20R
Connections:
- net +5V: no longer R1.2
- net GND: no longer C5.1, C7.1, SERVO0.1, SERVO1.1, SERVO10.1, SERVO11.1, SERVO2.1, SERVO3.1, SERVO4.1, SERVO5.1, SERVO6.1, SERVO7.1, SERVO8.1, SERVO9.1, SERVOX.1, SERVOY.1
- net N$17: no longer DEBUG.PP
- net N$18: now also SCL.TP; no longer SCL.MP
- net N$9: now also SDA.TP; no longer SDA.MP
- net UC_RESET: no longer R1.1
- net VSS: now also C5.1, C7.1, SERVO0.1, SERVO1.1, SERVO10.1, SERVO11.1, SERVO2.1, SERVO3.1, SERVO4.1, SERVO5.1, SERVO6.1, SERVO7.1, SERVO8.1, SERVO9.1, SERVOX.1, SERVOY.1

Commit message: Pcb, encore !
Parts:
- removed IC1: REG1117F, burr-brown:REG1117F
- removed RX, TX: SE14, solpad:SE14
- added IC4: LM2937, linear:LM2937
- added R1: (no value), resistor-shunt:PMD
- C3: value (none) -> 100nf
- C4: value (none) -> 10uf
Connections:
- removed net N$16: IC2.TX/RC6, TX.MP
- removed net N$17: IC2.RX/RC7, RX.MP
- new net RX_FROM_ARDUINO: IC2.TX/RC6, U1.D0
- new net TX_FROM_ARDUINO: IC2.RX/RC7, U1.D1
- net +5V: now also IC4.VO; no longer IC1.VOUT
- net VDD: now also IC4.VI, R1.2; no longer IC1.VIN
- net VEE: now also R1.1
- net VSS: now also IC4.GND; no longer IC1.GND
Other:
- note added: "Vérifier les condos nécessaires pour le régulateur"
Changed lines of the file:
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@@
 <setting verticaltext="up"/>
 </settings>
-<grid distance="0.1" unitdist="inch" unit="inch" style="lines" multiple="1" display="no" altdistance="0.01" altunitdist="inch" altunit="inch"/>
+<grid distance="0.1" unitdist="inch" unit="inch" style="dots" multiple="1" display="yes" altdistance="0.01" altunitdist="inch" altunit="inch"/>
 <layers>
 <layer number="1" name="Top" color="4" fill="1" visible="no" active="no"/>
@@
 <part name="IC2" library="microchip" deviceset="PIC16F87*" device="PT" technology="7" value="PIC18F452"/>
 <part name="SERVOX" library="con-lstb" deviceset="MA03-1" device=""/>
-<part name="C3" library="rcl" deviceset="C-EU" device="C1206"/>
-<part name="C4" library="rcl" deviceset="C-EU" device="C1206"/>
+<part name="C3" library="rcl" deviceset="C-EU" device="C1206" value="100nf"/>
+<part name="C4" library="rcl" deviceset="C-EU" device="C1206" value="10uf"/>
 <part name="SERVOY" library="con-lstb" deviceset="MA03-1" device=""/>
-<part name="RX" library="solpad" deviceset="SE14" device=""/>
-<part name="TX" library="solpad" deviceset="SE14" device=""/>
 <part name="C5" library="rcl" deviceset="C-EU" device="C1206"/>
 <part name="C7" library="rcl" deviceset="C-EU" device="C1206"/>
@@
 <part name="GND4" library="supply1" deviceset="GND" device=""/>
 <part name="GND8" library="supply1" deviceset="GND" device=""/>
-<part name="IC1" library="burr-brown" deviceset="REG1117" device="F"/>
 <part name="VSS3" library="supply1" deviceset="VSS" device=""/>
 <part name="VSS4" library="supply1" deviceset="VSS" device=""/>
@@
 <attribute name="TP_SIGNAL_NAME" value=""/>
 </part>
+<part name="R1" library="resistor-shunt" deviceset="PMD" device=""/>
+<part name="IC4" library="linear" deviceset="LM2937" device=""/>
 </parts>
 <sheets>
 <sheet>
 <plain>
+<text x="83.82" y="248.92" size="1.778" layer="91">Vérifier les condos nécessaires pour le régulateur</text>
 </plain>
 <instances>
@@
 <instance part="C4" gate="G$1" x="111.76" y="231.14"/>
 <instance part="SERVOY" gate="G$1" x="152.4" y="35.56" rot="R180"/>
-<instance part="RX" gate="1" x="134.62" y="152.4"/>
-<instance part="TX" gate="1" x="139.7" y="152.4"/>
 <instance part="C5" gate="G$1" x="66.04" y="73.66" rot="R90"/>
 <instance part="C7" gate="G$1" x="66.04" y="66.04" rot="R90"/>
@@
 <instance part="GND4" gate="1" x="274.32" y="137.16"/>
 <instance part="GND8" gate="1" x="264.16" y="43.18"/>
-<instance part="IC1" gate="G$1" x="96.52" y="236.22"/>
 <instance part="VSS3" gate="G$1" x="27.94" y="220.98"/>
 <instance part="VSS4" gate="G$1" x="81.28" y="220.98"/>
@@
 <attribute name="TP_SIGNAL_NAME" x="158.75" y="151.13" size="1.778" layer="97"/>
 </instance>
+<instance part="R1" gate="G$1" x="55.88" y="187.96"/>
+<instance part="IC4" gate="G$1" x="96.52" y="236.22"/>
 </instances>
 <busses>
@@
 <pinref part="VSS4" gate="G$1" pin="VSS"/>
 <wire x1="81.28" y1="226.06" x2="81.28" y2="223.52" width="0.1524" layer="91"/>
-</segment>
-<segment>
-<pinref part="IC1" gate="G$1" pin="GND"/>
-<pinref part="VSS5" gate="G$1" pin="VSS"/>
 </segment>
 <segment>
@@
 <pinref part="VSS21" gate="G$1" pin="VSS"/>
 </segment>
+<segment>
+<pinref part="VSS5" gate="G$1" pin="VSS"/>
+<pinref part="IC4" gate="G$1" pin="GND"/>
+<wire x1="96.52" y1="228.6" x2="96.52" y2="223.52" width="0.1524" layer="91"/>
+</segment>
 </net>
 <net name="N$25" class="0">
@@
 </segment>
 </net>
-<net name="N$16" class="0">
+<net name="RX_FROM_ARDUINO" class="0">
 <segment>
 <wire x1="132.08" y1="58.42" x2="139.7" y2="58.42" width="0.1524" layer="91"/>
 <wire x1="139.7" y1="58.42" x2="139.7" y2="149.86" width="0.1524" layer="91"/>
 <pinref part="IC2" gate="G$1" pin="TX/RC6"/>
-<pinref part="TX" gate="1" pin="MP"/>
-</segment>
-</net>
-<net name="N$17" class="0">
+<label x="139.7" y="152.4" size="1.778" layer="95" rot="R90"/>
+<junction x="139.7" y="149.86"/>
+</segment>
+<segment>
+<pinref part="U1" gate="G$1" pin="D0"/>
+<wire x1="294.64" y1="215.9" x2="294.64" y2="218.44" width="0.1524" layer="91"/>
+<junction x="294.64" y="218.44"/>
+<label x="294.64" y="220.98" size="1.778" layer="95" rot="R90"/>
+</segment>
+</net>
+<net name="TX_FROM_ARDUINO" class="0">
 <segment>
 <wire x1="132.08" y1="60.96" x2="134.62" y2="60.96" width="0.1524" layer="91"/>
 <wire x1="134.62" y1="149.86" x2="134.62" y2="60.96" width="0.1524" layer="91"/>
 <pinref part="IC2" gate="G$1" pin="RX/RC7"/>
-<pinref part="RX" gate="1" pin="MP"/>
+<junction x="134.62" y="149.86"/>
+<label x="134.62" y="152.4" size="1.778" layer="95" rot="R90"/>
+</segment>
+<segment>
+<pinref part="U1" gate="G$1" pin="D1"/>
+<wire x1="292.1" y1="215.9" x2="292.1" y2="218.44" width="0.1524" layer="91"/>
+<junction x="292.1" y="218.44"/>
+<label x="292.1" y="220.98" size="1.778" layer="95" rot="R90"/>
 </segment>
 </net>
@@
 </segment>
 <segment>
-<pinref part="IC1" gate="G$1" pin="VOUT"/>
-<wire x1="109.22" y1="236.22" x2="111.76" y2="236.22" width="0.1524" layer="91"/>
+<wire x1="106.68" y1="236.22" x2="111.76" y2="236.22" width="0.1524" layer="91"/>
 <wire x1="111.76" y1="236.22" x2="111.76" y2="238.76" width="0.1524" layer="91"/>
 <pinref part="C4" gate="G$1" pin="1"/>
@@
 <junction x="111.76" y="236.22"/>
 <pinref part="P+1" gate="1" pin="+5V"/>
+<pinref part="IC4" gate="G$1" pin="VO"/>
 </segment>
 <segment>
@@
 <net name="VDD" class="0">
 <segment>
-<pinref part="IC1" gate="G$1" pin="VIN"/>
 <pinref part="C3" gate="G$1" pin="1"/>
 <wire x1="48.26" y1="236.22" x2="81.28" y2="236.22" width="0.1524" layer="91"/>
-<wire x1="81.28" y1="236.22" x2="83.82" y2="236.22" width="0.1524" layer="91"/>
+<wire x1="81.28" y1="236.22" x2="86.36" y2="236.22" width="0.1524" layer="91"/>
 <wire x1="81.28" y1="236.22" x2="81.28" y2="233.68" width="0.1524" layer="91"/>
 <junction x="81.28" y="236.22"/>
@@
 <pinref part="VDD1" gate="G$1" pin="VDD"/>
 <wire x1="48.26" y1="236.22" x2="48.26" y2="238.76" width="0.1524" layer="91"/>
+<pinref part="IC4" gate="G$1" pin="VI"/>
 </segment>
 <segment>
@@
 <pinref part="IC3" gate="G$1" pin="R+"/>
 <wire x1="48.26" y1="187.96" x2="48.26" y2="185.42" width="0.1524" layer="91"/>
+<pinref part="R1" gate="G$1" pin="2"/>
+<wire x1="48.26" y1="187.96" x2="50.8" y2="187.96" width="0.1524" layer="91"/>
+<junction x="48.26" y="187.96"/>
 </segment>
 </net>
@@
 <pinref part="SUPPLY5" gate="G$1" pin="VEE"/>
 <wire x1="73.66" y1="187.96" x2="73.66" y2="190.5" width="0.1524" layer="91"/>
-</segment>
-</net>
+<pinref part="R1" gate="G$1" pin="1"/>
+<wire x1="60.96" y1="187.96" x2="63.5" y2="187.96" width="0.1524" layer="91"/>
+<junction x="63.5" y="187.96"/>
+</segment>
+</net>

Commit message: PCB
Parts:
- removed SV5: (no value), con-lstb:MA04-2
- added C1: 100nf, rcl:C-EUC1206
- added D1: MBRA340T3, diode:MBRA340T3
- added SV1: (no value), con-lstb:MA03-2
Connections:
- new net N$20: C4.1, D1.A, IC4.VO
- new net OPTION0: SV1.3, U1.A2
- new net OPTION1: SV1.5, U1.A3
- new net OPTION2: SV1.6, U1.A4/SDA
- new net OPTION3: SV1.4, U1.A5/SCL
- net +5V: now also C1.1, D1.C, SV1.1; no longer C4.1, IC4.VO, SV5.1
- net SWITCH0: no longer S2.S1
- net SWITCH1: no longer S3.S
- net VSS: now also C1.2, SV1.2; no longer SV5.2
Other:
- note removed: "Vérifier les condos nécessaires pour le régulateur"
- moved on the sheet: C4
