File: pcb/servo_controller.sch (EAGLE design)
At the start: 48 parts, among them IC2 PIC18F452, IC4 LM2937, U1 ARDUINOR3-DIMENSION

Commit message: PCB
Parts:
- added C2: (no value), rcl:CPOL-EUD
Connections:
- net VEE: now also C2.+
- net VSS: now also C2.-
Other:
- note added: "Ajouter un condo pour la sortie Servo"
- note added: "Vérifier la package de la résistance de mesure du courant"
Changed lines of the file:
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@@
 <setting verticaltext="up"/>
 </settings>
-<grid distance="0.1" unitdist="inch" unit="inch" style="lines" multiple="1" display="no" altdistance="0.01" altunitdist="inch" altunit="inch"/>
+<grid distance="0.1" unitdist="inch" unit="inch" style="dots" multiple="1" display="yes" altdistance="0.01" altunitdist="inch" altunit="inch"/>
 <layers>
 <layer number="1" name="Top" color="4" fill="1" visible="no" active="no"/>
@@
 <part name="VSS8" library="supply1" deviceset="VSS" device=""/>
 <part name="SV1" library="con-lstb" deviceset="MA03-2" device=""/>
+<part name="C2" library="rcl" deviceset="CPOL-EU" device="D"/>
+<part name="VSS22" library="supply1" deviceset="VSS" device=""/>
 </parts>
 <sheets>
 <sheet>
 <plain>
+<text x="99.06" y="264.16" size="5.08" layer="98" ratio="20">Ajouter un condo pour la sortie Servo</text>
+<text x="99.06" y="274.32" size="5.08" layer="98" ratio="20">Vérifier la package de la résistance de mesure du courant</text>
 </plain>
 <instances>
@@
 <instance part="VSS8" gate="G$1" x="27.94" y="160.02"/>
 <instance part="SV1" gate="1" x="187.96" y="170.18"/>
+<instance part="C2" gate="G$1" x="73.66" y="182.88"/>
+<instance part="VSS22" gate="G$1" x="73.66" y="172.72"/>
 </instances>
 <busses>
@@
 <wire x1="27.94" y1="162.56" x2="27.94" y2="165.1" width="0.1524" layer="91"/>
 </segment>
+<segment>
+<pinref part="C2" gate="G$1" pin="-"/>
+<pinref part="VSS22" gate="G$1" pin="VSS"/>
+<wire x1="73.66" y1="175.26" x2="73.66" y2="177.8" width="0.1524" layer="91"/>
+</segment>
 </net>
 <net name="N$25" class="0">
@@
 <wire x1="60.96" y1="187.96" x2="63.5" y2="187.96" width="0.1524" layer="91"/>
 <junction x="63.5" y="187.96"/>
+<pinref part="C2" gate="G$1" pin="+"/>
+<wire x1="73.66" y1="187.96" x2="73.66" y2="185.42" width="0.1524" layer="91"/>
+<junction x="73.66" y="187.96"/>
 </segment>
 </net>
@@
 <segment>
 <pinref part="IC3" gate="G$1" pin="VOUT"/>
-<wire x1="71.12" y1="170.18" x2="73.66" y2="170.18" width="0.1524" layer="91"/>
-<junction x="73.66" y="170.18"/>
-<label x="76.2" y="170.18" size="1.778" layer="95"/>
-</segment>
-<segment>
+<wire x1="71.12" y1="170.18" x2="78.74" y2="170.18" width="0.1524" layer="91"/>
+<junction x="78.74" y="170.18"/>
+<label x="81.28" y="170.18" size="1.778" layer="95"/>
+</segment>
+<segment>
