File: pcb/servo_controller.sch (EAGLE design)
At the start: 49 parts, among them IC2 PIC18F452, IC4 LM2937, U1 ARDUINOR3-DIMENSION

Commit message: PCB
Parts:
- removed R1: (no value), resistor-shunt:PMD
- added RSENSE: (no value), rcl:R-EU_R4527
Connections:
- net VDD: now also RSENSE.1; no longer R1.2
- net VEE: now also RSENSE.2; no longer R1.1
Changed lines of the file:
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@@
 <attribute name="TP_SIGNAL_NAME" value=""/>
 </part>
-<part name="R1" library="resistor-shunt" deviceset="PMD" device=""/>
 <part name="IC4" library="linear" deviceset="LM2937" device=""/>
 <part name="D1" library="diode" deviceset="MBRA340T3" device=""/>
@@
 <part name="C2" library="rcl" deviceset="CPOL-EU" device="D"/>
 <part name="VSS22" library="supply1" deviceset="VSS" device=""/>
+<part name="RSENSE" library="rcl" deviceset="R-EU_" device="R4527"/>
 </parts>
 <sheets>
@@
 <attribute name="TP_SIGNAL_NAME" x="158.75" y="151.13" size="1.778" layer="97"/>
 </instance>
-<instance part="R1" gate="G$1" x="55.88" y="187.96"/>
 <instance part="IC4" gate="G$1" x="96.52" y="236.22"/>
 <instance part="D1" gate="G$1" x="114.3" y="236.22"/>
@@
 <instance part="C2" gate="G$1" x="73.66" y="182.88"/>
 <instance part="VSS22" gate="G$1" x="73.66" y="172.72"/>
+<instance part="RSENSE" gate="G$1" x="55.88" y="187.96"/>
 </instances>
 <busses>
@@
 <pinref part="IC3" gate="G$1" pin="R+"/>
 <wire x1="48.26" y1="187.96" x2="48.26" y2="185.42" width="0.1524" layer="91"/>
-<pinref part="R1" gate="G$1" pin="2"/>
 <wire x1="48.26" y1="187.96" x2="50.8" y2="187.96" width="0.1524" layer="91"/>
 <junction x="48.26" y="187.96"/>
+<pinref part="RSENSE" gate="G$1" pin="1"/>
 </segment>
 </net>
@@
 <pinref part="SUPPLY5" gate="G$1" pin="VEE"/>
 <wire x1="73.66" y1="187.96" x2="73.66" y2="190.5" width="0.1524" layer="91"/>
-<pinref part="R1" gate="G$1" pin="1"/>
 <wire x1="60.96" y1="187.96" x2="63.5" y2="187.96" width="0.1524" layer="91"/>
 <junction x="63.5" y="187.96"/>
@@
 <wire x1="73.66" y1="187.96" x2="73.66" y2="185.42" width="0.1524" layer="91"/>
 <junction x="73.66" y="187.96"/>
-</segment>
-</net>
+<pinref part="RSENSE" gate="G$1" pin="2"/>
+</segment>
+</net>

Commit message: PCB Version 1.0.0
Parts:
- added C6: (no value), rcl:CPOL-EUD
Connections:
- net VEE: now also C6.+
- net VSS: now also C6.-
Other:
- note added: "Bleuette"
- note added: "Current probe"
- note added: "Interface"
- note added: "Power"
- note added: "Servo controller"
- note added: "Shield"
- note removed: "Ajouter un condo pour la sortie Servo"
- note removed: "Vérifier la package de la résistance de mesure du courant"
- moved on the sheet: C1, C2, C3, C4, C5, C7, C8, D1, IC2, IC3, IC4, LED1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

Commit message: Rev. 1.0.2, gerber file generation
Parts:
- removed IC4: LM2937, linear:LM2937
- removed LED2: (no value), led:LEDCHIPLED_0805
- removed LIPO+, LIPO-: SE14, solpad:SE14
- removed R7: (no value), rcl:R-EU_M0805
- removed S3: (no value), switch-omron:10-XX
- added IC1: PIC18F452, microchip:PIC16F877PT
- added LED0: (no value), led:LEDCHIPLED_0805
- added R1: (no value), rcl:R-EU_M1206
- added SP: (no value), switch:255SB
- added X1: (no value), con-wago-500:W237-102
- C2: value (none) -> 10uf; device rcl:CPOL-EUD -> rcl:C-EUC1206
- C4: value 10uf -> (none); device rcl:C-EUC1206 -> rcl:CPOL-EUD
- C5: device rcl:C-EUC1206 -> rcl:CPOL-EUD
- C6: device rcl:CPOL-EUD -> rcl:C-EUC1206
- IC2: value PIC18F452 -> LM2936MP-3.0; device microchip:PIC16F877PT -> national-semiconductor:LM2936MP-3.0
- R3: device rcl:R-EU_M1206 -> rcl:R-EU_M0805
- S1: device switch:255SB -> switch-omron:10-XX
- renumbered S2 to S0, SERVO0 to SRV0, SERVO1 to SRV1, SERVO10 to SRV10, SERVO11 to SRV11, SERVO2 to SRV2, SERVO3 to SRV3, SERVO4 to SRV4, SERVO5 to SRV5, SERVO6 to SRV6, SERVO7 to SRV7, SERVO8 to SRV8, SERVO9 to SRV9, SERVOX to SRVX, SERVOY to SRVY
Connections:
- removed net N$8 (its old number): LED2.A, R5.2
- new net N$7: LED0.A, R3.2
- net +5V: now also C3.1, C6.1, IC1.VDD, IC1.VDD@1, R5.2; no longer C1.1, C8.1, IC2.VDD, IC2.VDD@1, R7.2
- net LED0: now also LED0.C; no longer LED1.C
- net LED1: now also LED1.C; no longer LED2.C
- net LIPO_VOLTAGE: now also R1.1, R2.2; no longer R2.1, R3.2
- net N$1: now also IC1.RA0/AN0; no longer IC2.RA0/AN0
- net N$10: now also IC1.INT/RB0; no longer IC2.INT/RB0
- net N$11: now also IC1.RB1; no longer IC2.RB1
- net N$12: now also IC1.RB2; no longer IC2.RB2
- net N$13: now also IC1.PGM/RB3; no longer IC2.PGM/RB3
- net N$14: now also IC1.RB4; no longer IC2.RB4
- net N$15: now also SP.P, X1-2.KL; no longer LIPO+.MP, S1.P
- net N$18: now also IC1.RC3/SCK; no longer IC2.RC3/SCK
- net N$19: now also IC1.RD0/PSP0; no longer IC2.RD0/PSP0
- net N$2: now also IC1.RA1/AN1; no longer IC2.RA1/AN1
- net N$20: now also C2.1, IC2.VO; no longer C4.1, IC4.VO
- net N$22: now also IC1.PGD/RB7; no longer IC2.PGD/RB7
- net N$23: now also IC1.PGC/RB6; no longer IC2.PGC/RB6
- net N$24: now also IC1.RD1/PSP1; no longer IC2.RD1/PSP1
- net N$25: now also C8.2, IC1.OSC2/CLKOUT; no longer C7.2, IC2.OSC2/CLKOUT
- net N$27: now also C7.2, IC1.OSC1/CLKIN; no longer C5.2, IC2.OSC1/CLKIN
- net N$3: now also IC1.RA2/AN2; no longer IC2.RA2/AN2
- net N$32: now also IC1.RB5; no longer IC2.RB5
- net N$4: now also IC1.RA3/AN3; no longer IC2.RA3/AN3
- net N$5: now also IC1.RA4/T0CKI; no longer IC2.RA4/T0CKI
- net N$6: now also IC1.RC0/T1OSO; no longer IC2.RC0/T1OSO
- net N$9: now also IC1.SDI/RC4; no longer IC2.SDI/RC4
- net RX_FROM_ARDUINO: now also IC1.TX/RC6; no longer IC2.TX/RC6
- net SWITCH0: now also R6.1; no longer R7.1
- net SWITCH1: now also R5.1, S1.S1; no longer R6.1, S3.S1
- net TX_FROM_ARDUINO: now also IC1.RX/RC7; no longer IC2.RX/RC7
- net UC_RESET: now also IC1.!MCLR/THV; no longer IC2.!MCLR/THV
- net VDD: now also C1.1, IC2.VIN, R1.2, SP.O; no longer C3.1, IC4.VI, R2.2, S1.O
- net VEE: now also C4.+, C5.+; no longer C2.+, C6.+
- net VSS: now also C2.2, C4.-, C5.-, C6.2, C8.1, IC1.VSS, IC1.VSS@1, IC2.GND@1, IC2.GND@2, R2.1, S1.P, S1.P1, X1-1.KL; no longer C2.-, C4.2, C5.1, C6.-, C8.2, IC2.VSS, IC2.VSS@1, IC4.GND, LIPO-.MP, R5.1, S3.P, S3.P1
Other:
- moved on the sheet: C1, C3, C7, C8, LED1, R2, R3, R4, R5, R6

Commit message: Set values
Parts:
- C6: value (none) -> 100nf
- C7, C8: value (none) -> 22pf
- Q1: value (none) -> 10Mhz
- R1: value (none) -> 3.3k
- R2: value (none) -> 10k
- R3, R4: value (none) -> 1k
- R5, R6: value (none) -> 2.2k
Other:
- moved on the sheet: C1, C2, D1, IC2, R1, R2, SP

Commit message: Leg sensor + elec
Parts:
- RSENSE: value (none) -> 0.1
Changed lines of the file:
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@@
 <?xml version="1.0" encoding="utf-8"?>
 <!DOCTYPE eagle SYSTEM "eagle.dtd">
-<eagle version="6.2">
+<eagle version="6.4">
 <drawing>
 <settings>
@@
 <part name="C5" library="rcl" deviceset="CPOL-EU" device="D"/>
 <part name="VSS22" library="supply1" deviceset="VSS" device=""/>
-<part name="RSENSE" library="rcl" deviceset="R-EU_" device="R4527"/>
+<part name="RSENSE" library="rcl" deviceset="R-EU_" device="R4527" value="0.1"/>
 <part name="C4" library="rcl" deviceset="CPOL-EU" device="D"/>
 <part name="VSS23" library="supply1" deviceset="VSS" device=""/>
