File: pcb/sensor.sch (EAGLE design)
At the start: 9 parts, among them IC1 4512D, U1 ARDUINOR3-DIMENSION

Commit message: Sensor board
Parts:
- removed SV5: (no value), con-lsta:FE08-1
- added GY-27: (no value), con-lstb:MA05-1
- added JY-MCU: (no value), con-lstb:MA04-1
- added X1, X2: (no value), con-wago-500:W237-102
- SV1: device con-lstb:MA03-2 -> con-lstb:MA08-1W
- SV2: device con-lsta:FE08-1 -> con-lstb:MA08-1W
Connections:
- removed net N$13: U1.D5
- new net N$10: U1.D12
- new net N$11: U1.D7
- new net N$21: U1.D6
- new net N$8: U1.D13
- new net RXD: JY-MCU.1
- new net SCL: GY-27.4, U1.SCL
- new net SDA: GY-27.3, U1.SDA
- new net TXD: JY-MCU.2
- net +5V: now also C2.1, C3.1, GY-27.5, JY-MCU.4, SV1.3, SV1.5, SV1.7, U1.5V; no longer SV5.1, SV5.3, SV5.5, SV5.7
- net N$1: now also SV2.8; no longer SV5.8
- net N$2: now also SV1.2; no longer SV2.2
- net N$3: now also SV1.4; no longer SV2.4
- net N$4: now also SV2.6; no longer SV5.6
- net N$5: now also SV1.6; no longer SV2.6
- net N$6: now also SV1.8; no longer SV2.8
- net N$7: now also SV2.2; no longer SV5.2
- net N$9: now also SV2.4; no longer SV5.4
- net OUT: now also U1.D5
- net VSS: now also C2.2, C3.2, GY-27.1, IC1A.OE, JY-MCU.3, U1.GND, U1.GND1, U1.GND2, X1-2.KL, X2-2.KL; no longer SV1.2
Other:
- moved on the sheet: C1, C2, C3, IC1, IC1P, RN1

Commit message: Sensor board modif
Parts:
- removed X2: (no value), con-wago-500:W237-102
- added OUT: (no value), con-wago-500:W237-102
- added Q2: FDS5680, transistor-fet:FDS5680
- added R1: (no value), rcl:R-EU_M0805
- renumbered X1 to IN
Connections:
- removed net N$10: U1.D12
- removed net N$11: U1.D7
- removed net N$21: U1.D6
- new net +15V: IN-1.KL, OUT-1.KL
- new net N$13: OUT-2.KL, Q2.D
- new net POUT: Q2.G, R1.2, U1.D12
- net RXD: now also U1.D7
- net TXD: now also U1.D6
- net VSS: now also Q2.S, R1.1; no longer X2-2.KL
Changed lines of the file:
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@@
 <part name="P+7" library="supply1" deviceset="+5V" device=""/>
 <part name="VSS9" library="supply1" deviceset="VSS" device=""/>
-<part name="X1" library="con-wago-500" deviceset="W237-102" device=""/>
-<part name="X2" library="con-wago-500" deviceset="W237-102" device=""/>
+<part name="IN" library="con-wago-500" deviceset="W237-102" device=""/>
+<part name="OUT" library="con-wago-500" deviceset="W237-102" device=""/>
 <part name="VSS10" library="supply1" deviceset="VSS" device=""/>
 <part name="VSS11" library="supply1" deviceset="VSS" device=""/>
+<part name="Q2" library="transistor-fet" deviceset="FDS5680" device=""/>
+<part name="VSS12" library="supply1" deviceset="VSS" device=""/>
+<part name="R1" library="rcl" deviceset="R-EU_" device="M0805"/>
+<part name="VSS13" library="supply1" deviceset="VSS" device=""/>
+<part name="P+8" library="supply1" deviceset="+15V" device=""/>
+<part name="P+9" library="supply1" deviceset="+15V" device=""/>
 </parts>
 <sheets>
@@
 <attribute name="VALUE" x="152.4" y="109.22" size="1.778" layer="96" rot="R180"/>
 </instance>
-<instance part="X1" gate="-1" x="27.94" y="63.5"/>
-<instance part="X1" gate="-2" x="27.94" y="58.42"/>
-<instance part="X2" gate="-1" x="27.94" y="43.18"/>
-<instance part="X2" gate="-2" x="27.94" y="38.1"/>
-<instance part="VSS10" gate="G$1" x="35.56" y="53.34"/>
-<instance part="VSS11" gate="G$1" x="35.56" y="33.02"/>
+<instance part="IN" gate="-1" x="27.94" y="63.5"/>
+<instance part="IN" gate="-2" x="27.94" y="58.42"/>
+<instance part="OUT" gate="-1" x="27.94" y="35.56"/>
+<instance part="OUT" gate="-2" x="27.94" y="30.48"/>
+<instance part="VSS10" gate="G$1" x="101.6" y="45.72"/>
+<instance part="VSS11" gate="G$1" x="35.56" y="53.34"/>
+<instance part="Q2" gate="G$1" x="50.8" y="33.02" rot="R180"/>
+<instance part="VSS12" gate="G$1" x="43.18" y="17.78" smashed="yes">
+<attribute name="VALUE" x="45.72" y="15.24" size="1.778" layer="96" rot="R180"/>
+</instance>
+<instance part="R1" gate="G$1" x="58.42" y="27.94" rot="R90"/>
+<instance part="VSS13" gate="G$1" x="58.42" y="17.78" smashed="yes">
+<attribute name="VALUE" x="60.96" y="15.24" size="1.778" layer="96" rot="R180"/>
+</instance>
+<instance part="P+8" gate="1" x="35.56" y="68.58"/>
+<instance part="P+9" gate="1" x="35.56" y="40.64"/>
 </instances>
 <busses>
@@
 </segment>
 <segment>
-<pinref part="X2" gate="-2" pin="KL"/>
-<wire x1="33.02" y1="38.1" x2="35.56" y2="38.1" width="0.1524" layer="91"/>
+<pinref part="Q2" gate="G$1" pin="S"/>
+<wire x1="45.72" y1="35.56" x2="43.18" y2="35.56" width="0.1524" layer="91"/>
+<pinref part="VSS12" gate="G$1" pin="VSS"/>
+<wire x1="43.18" y1="35.56" x2="43.18" y2="20.32" width="0.1524" layer="91"/>
+</segment>
+<segment>
+<pinref part="R1" gate="G$1" pin="1"/>
+<pinref part="VSS13" gate="G$1" pin="VSS"/>
+<wire x1="58.42" y1="20.32" x2="58.42" y2="22.86" width="0.1524" layer="91"/>
+</segment>
+<segment>
+<pinref part="IN" gate="-2" pin="KL"/>
+<wire x1="33.02" y1="58.42" x2="35.56" y2="58.42" width="0.1524" layer="91"/>
 <pinref part="VSS11" gate="G$1" pin="VSS"/>
-<wire x1="35.56" y1="38.1" x2="35.56" y2="35.56" width="0.1524" layer="91"/>
-</segment>
-<segment>
-<pinref part="X1" gate="-2" pin="KL"/>
-<wire x1="33.02" y1="58.42" x2="35.56" y2="58.42" width="0.1524" layer="91"/>
-<pinref part="VSS10" gate="G$1" pin="VSS"/>
 <wire x1="35.56" y1="58.42" x2="35.56" y2="55.88" width="0.1524" layer="91"/>
 </segment>
@@
 </segment>
 </net>
-<net name="N$10" class="0">
-<segment>
-<pinref part="U1" gate="G$1" pin="D12"/>
-<wire x1="203.2" y1="154.94" x2="203.2" y2="157.48" width="0.1524" layer="91"/>
-<junction x="203.2" y="157.48"/>
-</segment>
-</net>
-<net name="N$11" class="0">
-<segment>
-<pinref part="U1" gate="G$1" pin="D7"/>
-<wire x1="218.44" y1="154.94" x2="218.44" y2="157.48" width="0.1524" layer="91"/>
-<junction x="218.44" y="157.48"/>
-</segment>
-</net>
-<net name="N$21" class="0">
-<segment>
-<pinref part="U1" gate="G$1" pin="D6"/>
-<wire x1="220.98" y1="154.94" x2="220.98" y2="157.48" width="0.1524" layer="91"/>
-<junction x="220.98" y="157.48"/>
-</segment>
-</net>
 <net name="SDA" class="0">
 <segment>
@@
 <label x="139.7" y="121.92" size="1.778" layer="95"/>
 </segment>
+<segment>
+<pinref part="U1" gate="G$1" pin="D6"/>
+<wire x1="220.98" y1="154.94" x2="220.98" y2="157.48" width="0.1524" layer="91"/>
+<junction x="220.98" y="157.48"/>
+<label x="220.98" y="160.02" size="1.778" layer="95" rot="R90"/>
+</segment>
 </net>
 <net name="RXD" class="0">
@@
 <label x="139.7" y="119.38" size="1.778" layer="95"/>
 </segment>
-</net>
+<segment>
+<pinref part="U1" gate="G$1" pin="D7"/>
+<wire x1="218.44" y1="154.94" x2="218.44" y2="157.48" width="0.1524" layer="91"/>
+<junction x="218.44" y="157.48"/>
+<label x="218.44" y="160.02" size="1.778" layer="95" rot="R90"/>
+</segment>
+</net>
+<net name="POUT" class="0">
+<segment>
+<pinref part="Q2" gate="G$1" pin="G"/>
+<wire x1="55.88" y1="35.56" x2="58.42" y2="35.56" width="0.1524" layer="91"/>
+<pinref part="R1" gate="G$1" pin="2"/>
+<wire x1="58.42" y1="35.56" x2="63.5" y2="35.56" width="0.1524" layer="91"/>
+<wire x1="58.42" y1="35.56" x2="58.42" y2="33.02" width="0.1524" layer="91"/>
+<junction x="58.42" y="35.56"/>
+<junction x="63.5" y="35.56"/>
+<label x="71.12" y="38.1" size="1.778" layer="95" rot="R180"/>
+</segment>
+<segment>
+<pinref part="U1" gate="G$1" pin="D12"/>
+<wire x1="203.2" y1="154.94" x2="203.2" y2="157.48" width="0.1524" layer="91"/>
+<junction x="203.2" y="157.48"/>
+</segment>
+</net>
+<net name="+15V" class="0">
+<segment>
+<pinref part="P+8" gate="1" pin="+15V"/>
+<wire x1="35.56" y1="66.04" x2="35.56" y2="63.5" width="0.1524" layer="91"/>
+<pinref part="IN" gate="-1" pin="KL"/>
+<wire x1="35.56" y1="63.5" x2="33.02" y2="63.5" width="0.1524" layer="91"/>
+</segment>
+<segment>
+<pinref part="P+9" gate="1" pin="+15V"/>
+<wire x1="35.56" y1="38.1" x2="35.56" y2="35.56" width="0.1524" layer="91"/>
+<pinref part="OUT" gate="-1" pin="KL"/>
+<wire x1="35.56" y1="35.56" x2="33.02" y2="35.56" width="0.1524" layer="91"/>
+</segment>
+</net>
+<net name="N$13" class="0">
+<segment>
+<pinref part="OUT" gate="-2" pin="KL"/>
+<pinref part="Q2" gate="G$1" pin="D"/>
+<wire x1="33.02" y1="30.48" x2="45.72" y2="30.48" width="0.1524" layer="91"/>
+</segment>
+</net>

Commit message: Sensor board, simple face
Parts:
- removed IC1: 4512D, 45xx:4512D
- removed Q2: FDS5680, transistor-fet:FDS5680
- added IC2: 4512N, 45xx:4512N
- added Q1: BUZ10, transistor-fet:BUZ10
Connections:
- net +5V: now also IC2P.VDD; no longer IC1P.VDD
- net ADDRA: now also IC2A.A; no longer IC1A.A
- net ADDRB: now also IC2A.B; no longer IC1A.B
- net ADDRC: now also IC2A.C; no longer IC1A.C
- net N$1: now also IC2A.X4; no longer IC1A.X4
- net N$13: now also Q1.D; no longer Q2.D
- net N$2: now also IC2A.X3; no longer IC1A.X3
- net N$3: now also IC2A.X2; no longer IC1A.X2
- net N$4: now also IC2A.X5; no longer IC1A.X5
- net N$5: now also IC2A.X1; no longer IC1A.X1
- net N$6: now also IC2A.X0; no longer IC1A.X0
- net N$7: now also IC2A.X7; no longer IC1A.X7
- net N$9: now also IC2A.X6; no longer IC1A.X6
- net OUT: now also IC2A.Z; no longer IC1A.Z
- net POUT: now also Q1.G; no longer Q2.G
- net VSS: now also IC2A.INH, IC2A.OE, IC2P.VSS, Q1.S; no longer IC1A.INH, IC1A.OE, IC1P.VSS, Q2.S
Changed lines of the file:
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@@
 </classes>
 <parts>
-<part name="IC1" library="45xx" deviceset="4512" device="D"/>
 <part name="VSS1" library="supply1" deviceset="VSS" device=""/>
 <part name="VSS2" library="supply1" deviceset="VSS" device=""/>
@@
 <part name="VSS10" library="supply1" deviceset="VSS" device=""/>
 <part name="VSS11" library="supply1" deviceset="VSS" device=""/>
-<part name="Q2" library="transistor-fet" deviceset="FDS5680" device=""/>
 <part name="VSS12" library="supply1" deviceset="VSS" device=""/>
 <part name="R1" library="rcl" deviceset="R-EU_" device="M0805"/>
@@
 <part name="P+8" library="supply1" deviceset="+15V" device=""/>
 <part name="P+9" library="supply1" deviceset="+15V" device=""/>
+<part name="IC2" library="45xx" deviceset="4512" device="N"/>
+<part name="Q1" library="transistor-fet" deviceset="BUZ10" device=""/>
 </parts>
 <sheets>
@@
 </plain>
 <instances>
-<instance part="IC1" gate="A" x="86.36" y="121.92"/>
 <instance part="VSS1" gate="G$1" x="132.08" y="144.78" smashed="yes">
 <attribute name="VALUE" x="134.62" y="142.24" size="1.778" layer="96" rot="R180"/>
@@
 <attribute name="VALUE" x="134.62" y="167.64" size="1.778" layer="96" rot="R180"/>
 </instance>
-<instance part="IC1" gate="P" x="83.82" y="162.56" rot="R90"/>
 <instance part="VSS3" gate="G$1" x="93.98" y="147.32"/>
 <instance part="P+2" gate="1" x="73.66" y="167.64"/>
@@
 <instance part="VSS10" gate="G$1" x="101.6" y="45.72"/>
 <instance part="VSS11" gate="G$1" x="35.56" y="53.34"/>
-<instance part="Q2" gate="G$1" x="50.8" y="33.02" rot="R180"/>
 <instance part="VSS12" gate="G$1" x="43.18" y="17.78" smashed="yes">
 <attribute name="VALUE" x="45.72" y="15.24" size="1.778" layer="96" rot="R180"/>
@@
 <instance part="P+8" gate="1" x="35.56" y="68.58"/>
 <instance part="P+9" gate="1" x="35.56" y="40.64"/>
+<instance part="IC2" gate="A" x="86.36" y="121.92"/>
+<instance part="IC2" gate="P" x="83.82" y="162.56" rot="R90"/>
+<instance part="Q1" gate="G$1" x="50.8" y="33.02" rot="R180"/>
 </instances>
 <busses>
@@
 <net name="+5V" class="0">
 <segment>
-<pinref part="IC1" gate="P" pin="VDD"/>
 <wire x1="76.2" y1="162.56" x2="73.66" y2="162.56" width="0.1524" layer="91"/>
 <pinref part="P+2" gate="1" pin="+5V"/>
@@
 <wire x1="73.66" y1="154.94" x2="78.74" y2="154.94" width="0.1524" layer="91"/>
 <junction x="73.66" y="162.56"/>
+<pinref part="IC2" gate="P" pin="VDD"/>
 </segment>
 <segment>
@@
 <net name="VSS" class="0">
 <segment>
-<pinref part="IC1" gate="P" pin="VSS"/>
 <pinref part="VSS3" gate="G$1" pin="VSS"/>
 <wire x1="91.44" y1="162.56" x2="93.98" y2="162.56" width="0.1524" layer="91"/>
@@
 <wire x1="86.36" y1="154.94" x2="93.98" y2="154.94" width="0.1524" layer="91"/>
 <junction x="93.98" y="154.94"/>
-</segment>
-<segment>
-<pinref part="IC1" gate="A" pin="INH"/>
+<pinref part="IC2" gate="P" pin="VSS"/>
+</segment>
+<segment>
 <wire x1="73.66" y1="104.14" x2="71.12" y2="104.14" width="0.1524" layer="91"/>
 <pinref part="VSS6" gate="G$1" pin="VSS"/>
 <wire x1="71.12" y1="104.14" x2="71.12" y2="101.6" width="0.1524" layer="91"/>
-<pinref part="IC1" gate="A" pin="OE"/>
 <wire x1="73.66" y1="106.68" x2="71.12" y2="106.68" width="0.1524" layer="91"/>
 <wire x1="71.12" y1="106.68" x2="71.12" y2="104.14" width="0.1524" layer="91"/>
 <junction x="71.12" y="104.14"/>
+<pinref part="IC2" gate="A" pin="INH"/>
+<pinref part="IC2" gate="A" pin="OE"/>
 </segment>
 <segment>
@@
 </segment>
 <segment>
-<pinref part="Q2" gate="G$1" pin="S"/>
 <wire x1="45.72" y1="35.56" x2="43.18" y2="35.56" width="0.1524" layer="91"/>
 <pinref part="VSS12" gate="G$1" pin="VSS"/>
 <wire x1="43.18" y1="35.56" x2="43.18" y2="20.32" width="0.1524" layer="91"/>
+<pinref part="Q1" gate="G$1" pin="S"/>
 </segment>
 <segment>
@@
 <segment>
 <wire x1="25.4" y1="116.84" x2="35.56" y2="116.84" width="0.1524" layer="91"/>
-<pinref part="IC1" gate="A" pin="X5"/>
 <wire x1="35.56" y1="116.84" x2="53.34" y2="116.84" width="0.1524" layer="91"/>
 <wire x1="53.34" y1="116.84" x2="53.34" y2="127" width="0.1524" layer="91"/>
@@
 <pinref part="RN1" gate="G$1" pin="7"/>
 <pinref part="SV2" gate="1" pin="6"/>
+<pinref part="IC2" gate="A" pin="X5"/>
 </segment>
 </net>
 <net name="N$1" class="0">
 <segment>
-<pinref part="IC1" gate="A" pin="X4"/>
 <wire x1="38.1" y1="121.92" x2="50.8" y2="121.92" width="0.1524" layer="91"/>
 <wire x1="50.8" y1="121.92" x2="50.8" y2="129.54" width="0.1524" layer="91"/>
@@
 <pinref part="RN1" gate="G$1" pin="6"/>
 <pinref part="SV2" gate="1" pin="8"/>
+<pinref part="IC2" gate="A" pin="X4"/>
 </segment>
 </net>
@@
 <wire x1="25.4" y1="137.16" x2="40.64" y2="137.16" width="0.1524" layer="91"/>
 <wire x1="40.64" y1="137.16" x2="40.64" y2="132.08" width="0.1524" layer="91"/>
-<pinref part="IC1" gate="A" pin="X3"/>
 <wire x1="40.64" y1="132.08" x2="73.66" y2="132.08" width="0.1524" layer="91"/>
 <wire x1="40.64" y1="104.14" x2="40.64" y2="132.08" width="0.1524" layer="91"/>
@@
 <pinref part="RN1" gate="G$1" pin="5"/>
 <pinref part="SV1" gate="1" pin="2"/>
+<pinref part="IC2" gate="A" pin="X3"/>
 </segment>
 </net>
 <net name="N$3" class="0">
 <segment>
-<pinref part="IC1" gate="A" pin="X2"/>
 <wire x1="73.66" y1="134.62" x2="43.18" y2="134.62" width="0.1524" layer="91"/>
 <wire x1="43.18" y1="134.62" x2="43.18" y2="142.24" width="0.1524" layer="91"/>
@@
 <pinref part="RN1" gate="G$1" pin="4"/>
 <pinref part="SV1" gate="1" pin="4"/>
+<pinref part="IC2" gate="A" pin="X2"/>
 </segment>
 </net>
@@
 <wire x1="25.4" y1="147.32" x2="45.72" y2="147.32" width="0.1524" layer="91"/>
 <wire x1="45.72" y1="147.32" x2="45.72" y2="137.16" width="0.1524" layer="91"/>
-<pinref part="IC1" gate="A" pin="X1"/>
 <wire x1="45.72" y1="137.16" x2="73.66" y2="137.16" width="0.1524" layer="91"/>
 <wire x1="45.72" y1="104.14" x2="45.72" y2="137.16" width="0.1524" layer="91"/>
@@
 <pinref part="RN1" gate="G$1" pin="3"/>
 <pinref part="SV1" gate="1" pin="6"/>
+<pinref part="IC2" gate="A" pin="X1"/>
 </segment>
 </net>
@@
 <wire x1="25.4" y1="152.4" x2="48.26" y2="152.4" width="0.1524" layer="91"/>
 <wire x1="48.26" y1="152.4" x2="48.26" y2="139.7" width="0.1524" layer="91"/>
-<pinref part="IC1" gate="A" pin="X0"/>
 <wire x1="73.66" y1="139.7" x2="48.26" y2="139.7" width="0.1524" layer="91"/>
 <wire x1="48.26" y1="139.7" x2="48.26" y2="104.14" width="0.1524" layer="91"/>
@@
 <pinref part="RN1" gate="G$1" pin="2"/>
 <pinref part="SV1" gate="1" pin="8"/>
+<pinref part="IC2" gate="A" pin="X0"/>
 </segment>
 </net>
 <net name="ADDRA" class="0">
 <segment>
-<pinref part="IC1" gate="A" pin="A"/>
 <wire x1="73.66" y1="116.84" x2="71.12" y2="116.84" width="0.1524" layer="91"/>
 <junction x="71.12" y="116.84"/>
 <label x="60.96" y="116.84" size="1.778" layer="95"/>
+<pinref part="IC2" gate="A" pin="A"/>
 </segment>
 <segment>
@@
 <net name="ADDRB" class="0">
 <segment>
-<pinref part="IC1" gate="A" pin="B"/>
 <wire x1="73.66" y1="114.3" x2="71.12" y2="114.3" width="0.1524" layer="91"/>
 <junction x="71.12" y="114.3"/>
 <label x="60.96" y="114.3" size="1.778" layer="95"/>
+<pinref part="IC2" gate="A" pin="B"/>
 </segment>
 <segment>
@@
 <net name="ADDRC" class="0">
 <segment>
-<pinref part="IC1" gate="A" pin="C"/>
 <wire x1="73.66" y1="111.76" x2="71.12" y2="111.76" width="0.1524" layer="91"/>
 <junction x="71.12" y="111.76"/>
 <label x="60.96" y="111.76" size="1.778" layer="95"/>
+<pinref part="IC2" gate="A" pin="C"/>
 </segment>
 <segment>
@@
 <wire x1="25.4" y1="111.76" x2="33.02" y2="111.76" width="0.1524" layer="91"/>
 <wire x1="33.02" y1="104.14" x2="33.02" y2="111.76" width="0.1524" layer="91"/>
-<pinref part="IC1" gate="A" pin="X6"/>
 <wire x1="33.02" y1="111.76" x2="55.88" y2="111.76" width="0.1524" layer="91"/>
 <wire x1="55.88" y1="111.76" x2="55.88" y2="124.46" width="0.1524" layer="91"/>
@@
 <pinref part="RN1" gate="G$1" pin="8"/>
 <pinref part="SV2" gate="1" pin="4"/>
+<pinref part="IC2" gate="A" pin="X6"/>
 </segment>
 </net>
 <net name="N$7" class="0">
 <segment>
-<pinref part="IC1" gate="A" pin="X7"/>
 <wire x1="73.66" y1="121.92" x2="58.42" y2="121.92" width="0.1524" layer="91"/>
 <wire x1="58.42" y1="121.92" x2="58.42" y2="106.68" width="0.1524" layer="91"/>
@@
 <pinref part="RN1" gate="G$1" pin="9"/>
 <pinref part="SV2" gate="1" pin="2"/>
+<pinref part="IC2" gate="A" pin="X7"/>
 </segment>
 </net>
 <net name="OUT" class="0">
 <segment>
-<pinref part="IC1" gate="A" pin="Z"/>
 <wire x1="99.06" y1="139.7" x2="104.14" y2="139.7" width="0.1524" layer="91"/>
 <junction x="104.14" y="139.7"/>
 <label x="106.68" y="139.7" size="1.778" layer="95"/>
+<pinref part="IC2" gate="A" pin="Z"/>
 </segment>
 <segment>
@@
 <net name="POUT" class="0">
 <segment>
-<pinref part="Q2" gate="G$1" pin="G"/>
 <wire x1="55.88" y1="35.56" x2="58.42" y2="35.56" width="0.1524" layer="91"/>
 <pinref part="R1" gate="G$1" pin="2"/>
@@
 <junction x="63.5" y="35.56"/>
 <label x="71.12" y="38.1" size="1.778" layer="95" rot="R180"/>
+<pinref part="Q1" gate="G$1" pin="G"/>
 </segment>
 <segment>
@@
 <segment>
 <pinref part="OUT" gate="-2" pin="KL"/>
-<pinref part="Q2" gate="G$1" pin="D"/>
 <wire x1="33.02" y1="30.48" x2="45.72" y2="30.48" width="0.1524" layer="91"/>
-</segment>
-</net>
+<pinref part="Q1" gate="G$1" pin="D"/>
+</segment>
+</net>
