File: pcb/sensor.brd (EAGLE design)
At the start: 68.6 x 53.3 mm, 9 parts, among them IC1 4512D, U1 ARDUINOR3-DIMENSION

Commit message: Sensor board
Parts:
- removed SV5: (no value), con-lsta:FE08
- added GY-27: (no value), con-lstb:MA05-1
- added JY-MCU: (no value), con-lstb:MA04-1
- added X1, X2: (no value), con-wago-500:W237-102
- SV1: device con-lstb:MA03-2 -> con-lstb:MA08-1W
- SV2: device con-lsta:FE08 -> con-lstb:MA08-1W
- moved RN1 95.3 mm to (15.2, 26.7), turned to 270 degrees
- moved SV2 67.3 mm to (10.2, 15.2), turned to 90 degrees
- moved SV1 46.0 mm to (10.2, 38.1), turned to 90 degrees
- moved C2 19.7 mm to (41.3, 32.4)
- moved IC1 7.96 mm to (24.1, 29.8)
- moved C3 7.18 mm to (24.1, 14.0)
- moved C1 6.84 mm to (24.1, 36.8)
Connections:
- removed net 5V: U1.5V
- removed net GND: U1.GND
- removed net GND1: U1.GND1
- removed net GND2: U1.GND2
- removed net N$13: U1.D5
- new net N$10: U1.D12
- new net N$11: U1.D7
- new net N$21: U1.D6
- new net N$8: U1.D13
- new net RXD: JY-MCU.1
- new net SCL: GY-27.4, U1.SCL
- new net SDA: GY-27.3, U1.SDA
- new net TXD: JY-MCU.2
- net +5V: now also C2.1, C3.1, GY-27.5, JY-MCU.4, SV1.3, SV1.5, SV1.7, U1.5V; no longer SV5.1, SV5.3, SV5.5, SV5.7
- net N$1: now also SV2.8; no longer SV5.8
- net N$2: now also SV1.2; no longer SV2.2
- net N$3: now also SV1.4; no longer SV2.4
- net N$4: now also SV2.6; no longer SV5.6
- net N$5: now also SV1.6; no longer SV2.6
- net N$6: now also SV1.8; no longer SV2.8
- net N$7: now also SV2.2; no longer SV5.2
- net N$9: now also SV2.4; no longer SV5.4
- net OUT: now also U1.D5
- net VSS: now also C2.2, C3.2, GY-27.1, IC1.15, JY-MCU.3, U1.GND, U1.GND1, U1.GND2, X1.2, X2.2; no longer SV1.2
Routing:
- added copper zone on layer 1, net VSS

Commit message: Sensor board modif
Parts:
- removed X1, X2: (no value), con-wago-500:W237-102
- added IN, OUT: (no value), con-wago-500:W237-102
- added Q2: FDS5680, transistor-fet:SO-8
- added R1: (no value), rcl:M0805
- moved GY-27 24.7 mm to (29.2, 14.0)
- moved JY-MCU 24.1 mm to (31.1, 39.4)
- moved IC1 4.49 mm to (23.5, 25.4)
- moved RN1 0.63 mm to (15.9, 26.7)
- moved SV1 0.63 mm to (10.8, 38.1)
- moved SV2 0.63 mm to (10.8, 15.2)
Connections:
- removed net N$10: U1.D12
- removed net N$11: U1.D7
- removed net N$21: U1.D6
- new net +15V: IN.1, OUT.1
- new net N$13: OUT.2, Q2.5, Q2.6, Q2.7, Q2.8
- new net POUT: Q2.4, R1.2, U1.D12
- net RXD: now also U1.D7
- net TXD: now also U1.D6
- net VSS: now also IN.2, Q2.1, Q2.2, Q2.3, R1.1; no longer X1.2, X2.2

Commit message: Sensor board, simple face
Parts:
- removed IC1: 4512D, 45xx:SO16
- removed Q2: FDS5680, transistor-fet:SO-8
- added IC2: 4512N, 45xx:DIL16
- added Q1: BUZ10, transistor-fet:TO220
- moved C3 11.1 mm to (21.6, 3.17), turned to 180 degrees
- moved C1 8.54 mm to (29.8, 43.2), turned to 90 degrees
- moved R1 7.18 mm to (52.1, 8.89), turned to 0 degrees
- moved RN1 5.43 mm to (17.8, 31.8)
- moved JY-MCU 3.81 mm to (34.9, 39.4)
- moved C2 3.70 mm to (39.4, 35.6)
- moved GY-27 1.91 mm to (27.3, 14.0)
Connections:
- net +5V: now also IC2.16; no longer IC1.16
- net ADDRA: now also IC2.11; no longer IC1.11
- net ADDRB: now also IC2.12; no longer IC1.12
- net ADDRC: now also IC2.13; no longer IC1.13
- net N$1: now also IC2.5; no longer IC1.5
- net N$13: now also Q1.2; no longer Q2.5, Q2.6, Q2.7, Q2.8
- net N$2: now also IC2.4; no longer IC1.4
- net N$3: now also IC2.3; no longer IC1.3
- net N$4: now also IC2.6; no longer IC1.6
- net N$5: now also IC2.2; no longer IC1.2
- net N$6: now also IC2.1; no longer IC1.1
- net N$7: now also IC2.9; no longer IC1.9
- net N$9: now also IC2.7; no longer IC1.7
- net OUT: now also IC2.14; no longer IC1.14
- net POUT: now also Q1.1; no longer Q2.4
- net VSS: now also IC2.10, IC2.15, IC2.8, Q1.3; no longer IC1.10, IC1.15, IC1.8, Q2.1, Q2.2, Q2.3
Routing:
- net +5V: track 0.00 -> 97.4 mm
- net ADDRA: track 0.00 -> 49.9 mm
- net ADDRB: track 0.00 -> 46.4 mm
- net ADDRC: track 0.00 -> 43.0 mm
- net SCL: track 0.00 -> 41.8 mm
- net OUT: track 0.00 -> 39.0 mm
- net SDA: track 0.00 -> 32.6 mm
- net TXD: track 0.00 -> 22.4 mm
- net N$9: track 0.00 -> 20.1 mm
- net N$7: track 0.00 -> 18.9 mm
- net N$6: track 0.00 -> 17.9 mm
- net N$4: track 0.00 -> 17.6 mm
- net +15V: track 0.00 -> 17.6 mm
- net RXD: track 0.00 -> 17.3 mm
- net N$5: track 0.00 -> 15.0 mm
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
Commit message: Sensor board v1
Parts:
- moved C3 10.5 mm to (31.1, 7.62), turned to 90 degrees
- moved GY-27 2.54 mm to (27.3, 11.4)
- moved C1 2.13 mm to (30.8, 41.3), turned to 0 degrees
- moved R1 1.80 mm to (53.3, 7.62), turned to 90 degrees
Routing:
- net POUT: track 0.00 -> 60.6 mm
- net +5V: track 97.4 -> 143.2 mm, vias 0 -> 2
- net VSS: track 14.8 -> 58.7 mm, vias 0 -> 4
- net SDA: track 32.6 -> 48.0 mm
- net N$7: track 18.9 -> 33.5 mm, vias 0 -> 2
- net N$13: track 0.00 -> 10.3 mm
- net SCL: track 41.8 -> 51.8 mm
- net N$6: track 17.9 -> 16.4 mm
Other:
- board text added: "v1"
