File: pcb/servo_controller_pi.brd (EAGLE design)
At the start: 73 parts, among them IC1 PIC18F452, IC2 LM2936MP-5.0, IC3 MAX4173FESA+, IC4 LM2936MP-3.3, IC5 4512D, IC7 LM358D, Q1 10Mhz, Q2 BUZ10, Q4 BC848ALT1SMD

Commit message: Bleuette Pi
Parts:
- removed C13: 100nf, rcl:C1206
- removed C8: 22pf, rcl:C0805
- removed D1, D5: MBRA340T3, diode:SMA
- removed IC2: LM2936MP-5.0, national-semiconductor:SOT223
- removed IC7: LM358D, linear:SO08
- removed IN, OUT, X1: (no value), con-wago-500:W237-102
- removed Q2: BUZ10, transistor-fet:TO220
- removed R8: (no value), rcl:M0805
- removed SCL, SDA: TPTP20R, testpad:TP20R
- removed SRVX, SRVY: (no value), con-lstb:MA03-1
- removed SV3: (no value), con-lstb:MA04-2
- added C14, C15: (no value), rcl:PANASONIC_A
- added C16: (no value), rcl:PANASONIC_B
- added C17: 100nf, rcl:C0805
- added IC6: LM386M-1, linear:SO08
- added P5V, PGND, PLIPO: (no value), wirepad:2,54/0,8
- added R15: (no value), pot:3223J
- added R3: (no value), rcl:M0805
- added SV4, SX, SY: (no value), con-lstb:MA03-1
- added SV5: (no value), con-lstb:MA05-2
- C1: value 100nf -> (none); device rcl:C1206 -> rcl:PANASONIC_F
- C10, C11: value (none) -> 22pf
- C12: value 10uf -> (none); device rcl:C1206 -> rcl:C0805
- C2: value 10uf -> (none); device rcl:C1206 -> rcl:PANASONIC_F
- C4: value (none) -> 10uf; device rcl:PANASONIC_D -> rcl:C0805
- C5: value (none) -> 100nf; device rcl:PANASONIC_D -> rcl:C0805
- C6: value 100nf -> (none)
- C7: value 22pf -> 100nf
- C9: device rcl:PANASONIC_F -> rcl:PANASONIC_D
- moved C12 59.5 mm to (65.1, 24.1)
- moved C9 57.5 mm to (48.3, 4.76), turned to 90 degrees
- moved C4 45.2 mm to (13.0, 33.0)
- moved R12 39.7 mm to (33.3, 14.0)
- moved C11 32.6 mm to (38.1, 31.4)
- moved C6 30.5 mm to (67.6, 28.3), turned to 180 degrees
- moved C10 25.6 mm to (42.2, 31.4)
- moved C3 21.6 mm to (3.81, 32.4)
- moved LED-STRIP 19.2 mm to (81.9, 34.9)
- moved C5 18.3 mm to (3.17, 10.8), turned to 180 degrees
- moved C2 17.7 mm to (6.67, 44.5), turned to 0 degrees
- moved R14 15.9 mm to (21.0, 33.0), turned to 180 degrees
- moved LED2 15.6 mm to (17.1, 33.0), turned to 90 degrees
- moved C1 15.6 mm to (17.1, 20.3), turned to 180 degrees
- moved R1 14.5 mm to (10.8, 26.4)
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- renumbered SRV0 to S0, SRV1 to S1, SRV10 to S10, SRV11 to S11, SRV2 to S2, SRV3 to S3, SRV4 to S4, SRV5 to S5, SRV6 to S6, SRV7 to S7, SRV8 to S8, SRV9 to S9
Connections:
- removed net +15V: IN.1, OUT.1
- removed net N$18: IC1.37, SCL.TP
- removed net N$20: C2.1, D1.A, IC2.3
- removed net N$36: OUT.2, Q2.2
- removed net N$38: C12.1, D5.A, IC4.3
- removed net N$9: IC1.42, SDA.TP
- removed net POUT: Q2.1, R8.2, U$3.15
- removed net V+: IC7.8
- removed net V-: IC7.4
- new net N$40: C15.+, SV4.2
- new net N$41: IC6.3, R15.2
- new net N$42: C16.+, IC6.5, R3.2
- new net N$43: C17.1, R3.1
- new net N$7: C14.-, C15.-, R15.3
- new net N$8: C14.+, SV4.3
- new net OPTION4: SV5.5, U$3.15
- net +3V3: now also C12.1, C4.1, C6.1, IC4.3, SV5.9; no longer C10.1, C11.1, D5.C, SV3.1, U$3.1
- net +5V: now also C2.+, C5.1, C7.1, IC6.6, P5V.1, SV5.10, U$3.2; no longer C13.1, C6.1, C9.+, D1.C
- net N$19: now also SX.3; no longer SRVX.3
- net N$24: now also SY.3; no longer SRVY.3
- net N$25: now also C11.2; no longer C8.2
- net N$27: now also C10.2; no longer C7.2
- net OPTION0: now also SV5.1; no longer SV3.3
- net OPTION1: now also SV5.2; no longer SV3.4
- net OPTION2: now also SV5.3; no longer SV3.5
- net OPTION3: now also SV5.4; no longer SV3.6
- net SCL: now also SV5.8; no longer SV3.7
- net SDA: now also SV5.6; no longer SV3.8
- net VDD: now also C1.+, PLIPO.1; no longer C1.1, IC2.1, X1.2
- net VEE: now also C9.+, SX.2, SY.2; no longer C4.+, C5.+, SRVX.2, SRVY.2
- net VSS: now also C1.-, C10.1, C11.1, C17.2, C2.-, C4.2, C5.2, C7.2, IC6.2, IC6.4, PGND.1, R15.1, SV4.1, SV5.7, SX.1, SY.1; no longer C1.2, C10.2, C11.2, C13.2, C2.2, C4.-, C5.-, C7.1, C8.1, IC2.2, IC2.4, IN.2, Q2.3, R8.1, SRVX.1, SRVY.1, SV3.2, X1.1
Routing:
- net +3V3: track 61.4 -> 176.7 mm, vias 0 -> 2
- net SCL: track 0.00 -> 76.0 mm
- net +5V: track 28.9 -> 92.4 mm, vias 0 -> 1
- net N$35: track 10.2 -> 67.3 mm, vias 0 -> 1
- net SDA: track 0.00 -> 46.5 mm
- net LIPO_VOLTAGE: track 2.16 -> 43.3 mm, vias 0 -> 2
- net VSS: track 49.8 -> 87.0 mm, vias 6 -> 10
- net OPTION4: track 0.00 -> 23.5 mm
- net OPTION0: track 0.00 -> 20.6 mm
- net OPTION2: track 0.00 -> 20.3 mm
- net VEE: track 196.1 -> 178.2 mm
- net VDD: track 19.3 -> 33.4 mm
- net N$33: track 6.47 -> 20.6 mm
- net OPTION1: track 0.00 -> 12.3 mm
- net OPTION3: track 0.00 -> 11.2 mm
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Other:
- board text added: "0"
- board text added: "1"
- board text added: "2"
- board text added: "3"
- board text added: "4"
- board text added: "5"
- board text added: "6"
- board text added: "7"
- board text removed: "+"
