File: pcb/servo_controller_pi.sch (EAGLE design)
At the start: 109 parts, among them IC1 PIC18F452, IC2 DS1339, IC3 MAX4173FESA+, IC4 LM2936MP-3.3, IC6 LM386M-1, IC7 GY-27, IC8 MCP23017SO, Q1 10Mhz

Commit message: BleuettePi new modification
Parts:
- removed IC8: MCP23017SO, adafruit:MCP23017SO
- removed SV3: (no value), con-lstb:MA05-2
- added IC5: MCP23017SS, adafruit:MCP23017SS
- added X1: (no value), con-wago-500:W237-4
- SV1: device con-lstb:MA04-1 -> con-lstb:MA05-2
- SV2: device con-lstb:MA08-2 -> con-lstb:MA05-2
Connections:
- removed net OUT: U$3.12-GPIO1
- new net OPTION4: U$3.21-SPI-MISO
- net +5V: now also IC5.!RESET, IC5.VDD, SV1.10, SV2.10, X1-2.KL; no longer IC8.!RESET, IC8.VDD, SV1.2, SV3.10
- net +7V: now also X1-3.KL; no longer SV1.3
- net GPA0: now also IC5.GPA0, SV1.1; no longer IC8.GPA0, SV2.2
- net GPA1: now also IC5.GPA1, SV1.2; no longer IC8.GPA1, SV2.4
- net GPA2: now also IC5.GPA2, SV1.3; no longer IC8.GPA2, SV2.6
- net GPA3: now also IC5.GPA3, SV1.4; no longer IC8.GPA3, SV2.8
- net GPA4: now also IC5.GPA4, SV1.5; no longer IC8.GPA4, SV2.10
- net GPA5: now also IC5.GPA5, SV1.6; no longer IC8.GPA5, SV2.12
- net GPA6: now also IC5.GPA6, SV1.7; no longer IC8.GPA6, SV2.14
- net GPA7: now also IC5.GPA7, SV1.8; no longer IC8.GPA7, SV2.16
- net GPB0: now also IC5.GPB0, SV2.1; no longer IC8.GPB0, SV3.2
- net GPB1: now also IC5.GPB1, SV2.2; no longer IC8.GPB1, SV3.1
- net GPB2: now also IC5.GPB2, SV2.3; no longer IC8.GPB2, SV3.4
- net GPB3: now also IC5.GPB3, SV2.4; no longer IC8.GPB3, SV3.3
- net GPB4: now also IC5.GPB4, SV2.5; no longer IC8.GPB4, SV3.6
- net GPB5: now also IC5.GPB5, SV2.6; no longer IC8.GPB5, SV3.5
- net GPB6: now also IC5.GPB6, SV2.7; no longer IC8.GPB6, SV3.8
- net GPB7: now also DRDY.1, IC5.GPB7, SV2.8; no longer IC8.GPB7, SV3.7
- net INTA: now also IC5.INTA; no longer IC8.INTA
- net INTB: now also IC5.INTB; no longer IC8.INTB
- net INTD: now also U$3.12-GPIO1; no longer DRDY.1
- net OPTION2: now also U$3.13-GPIO2; no longer U$3.16-GPIO4
- net OPTION3: now also U$3.15-GPIO3; no longer U$3.13-GPIO2
- net SCL: now also IC5.SCL; no longer IC8.SCL
- net SDA: now also IC5.SDA; no longer IC8.SDA
- net TRIGGER: now also U$3.16-GPIO4; no longer U$3.15-GPIO3
- net VDD: now also X1-4.KL; no longer SV1.4
- net VSS: now also IC5.A0, IC5.A1, IC5.A2, IC5.VSS, SV1.9, X1-1.KL; no longer IC8.A0, IC8.A1, IC8.A2, IC8.VSS, SV1.1, SV2.1, SV2.11, SV2.13, SV2.15, SV2.3, SV2.5, SV2.7, SV3.9
Other:
- note added: "INTD : Interrupt from PIC"
- note added: "Real Time Clock"
- note removed: "INTD : Interrupt from PIC <- CONNECT ME !"
- note removed: "J_VOLT : Battery voltage read by MCP or PIC"
- moved on the sheet: C5, C6, D1, IC2, IC3, PWR, Q6, R14, R19, R6, R8, RSENSE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
